Commit message: Remove unused material "opaque2550255" and add new material "steel_satin" with a gray color in materials.xacro for humanoid right leg description.

File: humanoidrightleg_description/urdf/humanoidrightleg.xacro (robot description, xacro)
@@ -5,7 +5,7 @@
 <link name="base_link">
   <inertial>
-    <origin xyz="-0.191552173924666 0.380845062266963 -0.172380256596757" rpy="0 0 0"/>
-    <mass value="0.0688919713115792"/>
-    <inertia ixx="8.05202310847145e-06" iyy="1.41808431909076e-05" izz="2.19458145304646e-05" ixy="-3.30654655814576e-07" iyz="-8.626208601592023e-11" ixz="-3.62199873999575e-09"/>
+    <origin xyz="-2.137404171899072e-14 0 0.005" rpy="0 0 0"/>
+    <mass value="0.15083462441733"/>
+    <inertia ixx="2.21517549468842e-05" iyy="3.39267549369311e-05" izz="5.35645994768598e-05" ixy="0" iyz="0" ixz="3.081487911019577e-33"/>
   </inertial>
   <visual>
@@ -14,5 +14,5 @@
       <mesh filename="package://humanoidrightleg_description/meshes/base_link.stl" scale="0.001 0.001 0.001"/>
     </geometry>
-    <material name="opaque2550255"/>
+    <material name="steel_satin"/>
   </visual>
   <collision>
@@ -23,12 +23,2192 @@
   </collision>
 </link>
+<link name="RMD-X10-S2_MIR4__3_Stator_1">
+  <inertial>
+    <origin xyz="-1.1561410892626987e-08 0.0007996823934559865 0.03182069992246948" rpy="0 0 0"/>
+    <mass value="1.55306904844425"/>
+    <inertia ixx="0.00285644715024274" iyy="0.00292757747778099" izz="0.00369780684183897" ixy="7.224771163531730e-11" iyz="1.67010427996743e-05" ixz="4.91373014642689e-10"/>
+  </inertial>
+  <visual>
+    <origin xyz="-0.0 -0.0 -0.01" rpy="0 0 0"/>
+    <geometry>
+      <mesh filename="package://humanoidrightleg_description/meshes/RMD-X10-S2_MIR4__3_Stator_1.stl" scale="0.001 0.001 0.001"/>
+    </geometry>
+    <material name="opaque727161"/>
+  </visual>
+  <collision>
+    <origin xyz="-0.0 -0.0 -0.01" rpy="0 0 0"/>
+    <geometry>
+      <mesh filename="package://humanoidrightleg_description/meshes/RMD-X10-S2_MIR4__3_Stator_1.stl" scale="0.001 0.001 0.001"/>
+    </geometry>
+  </collision>
+</link>
+<link name="leg-pitch-elastic__1__1">
+  <inertial>
+    <origin xyz="0.0043331749249106155 0.00111244839801433 0.028315467914110406" rpy="0 0 0"/>
+    <mass value="0.0245291042760104"/>
+    <inertia ixx="9.8175039693855e-06" iyy="8.21623306395601e-06" izz="2.92015853283537e-06" ixy="4.21998763905152e-07" iyz="-2.69850308691085e-07" ixz="9.97190866763669e-08"/>
+  </inertial>
+  <visual>
+    <origin xyz="0.071138 0.011355 -0.012" rpy="0 0 0"/>
+    <geometry>
+      <mesh filename="package://humanoidrightleg_description/meshes/leg-pitch-elastic__1__1.stl" scale="0.001 0.001 0.001"/>
+    </geometry>
+    <material name="opaque191191191"/>
+  </visual>
+  <collision>
+    <origin xyz="0.071138 0.011355 -0.012" rpy="0 0 0"/>
+    <geometry>
+      <mesh filename="package://humanoidrightleg_description/meshes/leg-pitch-elastic__1__1.stl" scale="0.001 0.001 0.001"/>
+    </geometry>
+  </collision>
+</link>
+<link name="leg-pitch-elastic__3__1">
+  <inertial>
+    <origin xyz="0.00028161841037692426 -0.004464786595415545 0.030684539200331342" rpy="0 0 0"/>
+    <mass value="0.0245291042760104"/>
+    <inertia ixx="8.121096179216e-06" iyy="9.91264085412532e-06" izz="2.9201585328353e-06" ixy="-1.2919753996385e-07" iyz="1.1450155860264e-08" ixz="-2.87457786952056e-07"/>
+  </inertial>
+  <visual>
+    <origin xyz="0.082894 0.027535 -0.012" rpy="0 0 0"/>
+    <geometry>
+      <mesh filename="package://humanoidrightleg_description/meshes/leg-pitch-elastic__3__1.stl" scale="0.001 0.001 0.001"/>
+    </geometry>
+    <material name="opaque191191191"/>
+  </visual>
+  <collision>
+    <origin xyz="0.082894 0.027535 -0.012" rpy="0 0 0"/>
+    <geometry>
+      <mesh filename="package://humanoidrightleg_description/meshes/leg-pitch-elastic__3__1.stl" scale="0.001 0.001 0.001"/>
+    </geometry>
+  </collision>
+</link>
+<link name="leg-pitch-elastic__2__1">
+  <inertial>
+    <origin xyz="-0.000281419190083107 0.004464713281593341 0.030684532085865125" rpy="0 0 0"/>
+    <mass value="0.0245291042760104"/>
+    <inertia ixx="8.12109617921613e-06" iyy="9.9126408541253e-06" izz="2.92015853283526e-06" ixy="-1.29197539963853e-07" iyz="-1.14501558602572e-08" ixz="2.87457786951236e-07"/>
+  </inertial>
+  <visual>
+    <origin xyz="-0.011184 0.071165 -0.012" rpy="0 0 0"/>
+    <geometry>
+      <mesh filename="package://humanoidrightleg_description/meshes/leg-pitch-elastic__2__1.stl" scale="0.001 0.001 0.001"/>
+    </geometry>
+    <material name="opaque191191191"/>
+  </visual>
+  <collision>
+    <origin xyz="-0.011184 0.071165 -0.012" rpy="0 0 0"/>
+    <geometry>
+      <mesh filename="package://humanoidrightleg_description/meshes/leg-pitch-elastic__2__1.stl" scale="0.001 0.001 0.001"/>
+    </geometry>
+  </collision>
+</link>
+<link name="leg-pitch-elastic_1">
+  <inertial>
+    <origin xyz="-0.00433297570461362 -0.0011125217118188452 0.02831546079961827" rpy="0 0 0"/>
+    <mass value="0.0245291042760104"/>
+    <inertia ixx="9.81750396938545e-06" iyy="8.21623306395594e-06" izz="2.92015853283533e-06" ixy="4.21998763905183e-07" iyz="2.69850308691019e-07" ixz="-9.97190866774748e-08"/>
+  </inertial>
+  <visual>
+    <origin xyz="0.000572 0.087345 -0.012" rpy="0 0 0"/>
+    <geometry>
+      <mesh filename="package://humanoidrightleg_description/meshes/leg-pitch-elastic_1.stl" scale="0.001 0.001 0.001"/>
+    </geometry>
+    <material name="opaque191191191"/>
+  </visual>
+  <collision>
+    <origin xyz="0.000572 0.087345 -0.012" rpy="0 0 0"/>
+    <geometry>
+      <mesh filename="package://humanoidrightleg_description/meshes/leg-pitch-elastic_1.stl" scale="0.001 0.001 0.001"/>
+    </geometry>
+  </collision>
+</link>
+<link name="hip-motor-bracket-v5-right_MIR_1">
+  <inertial>
+    <origin xyz="0.017145099610158858 -0.04935003665687157 -0.004500000000001279" rpy="0 0 0"/>
+    <mass value="0.0629963904640038"/>
+    <inertia ixx="4.19044655038384e-05" iyy="6.2878187218024e-05" izz="0.000103932201450599" ixy="3.22752390165202e-05" iyz="-2.286988957586611e-18" ixz="4.397795062144327e-18"/>
+  </inertial>
+  <visual>
+    <origin xyz="0.053 0.0 -0.012" rpy="0 0 0"/>
+    <geometry>
+      <mesh filename="package://humanoidrightleg_description/meshes/hip-motor-bracket-v5-right_MIR_1.stl" scale="0.001 0.001 0.001"/>
+    </geometry>
+    <material name="opaque245245245"/>
+  </visual>
+  <collision>
+    <origin xyz="0.053 0.0 -0.012" rpy="0 0 0"/>
+    <geometry>
+      <mesh filename="package://humanoidrightleg_description/meshes/hip-motor-bracket-v5-right_MIR_1.stl" scale="0.001 0.001 0.001"/>
+    </geometry>
+  </collision>
+</link>
+<link name="innner-thigh-magnet-encoder__1__1">
+  <inertial>
+    <origin xyz="0.018384650368951743 -0.002568109841095942 -0.02778155630905323" rpy="0 0 0"/>
+    <mass value="0.0278904055568687"/>
+    <inertia ixx="1.76659445346298e-05" iyy="1.5985340031158e-05" izz="1.10005716364315e-05" ixy="-2.56247035072647e-06" iyz="6.12320058242576e-06" ixz="4.44219697098464e-06"/>
+  </inertial>
+  <visual>
+    <origin xyz="0.042878 0.031153 -0.003" rpy="0 0 0"/>
+    <geometry>
+      <mesh filename="package://humanoidrightleg_description/meshes/innner-thigh-magnet-encoder__1__1.stl" scale="0.001 0.001 0.001"/>
+    </geometry>
+    <material name="opaque191191191"/>
+  </visual>
+  <collision>
+    <origin xyz="0.042878 0.031153 -0.003" rpy="0 0 0"/>
+    <geometry>
+      <mesh filename="package://humanoidrightleg_description/meshes/innner-thigh-magnet-encoder__1__1.stl" scale="0.001 0.001 0.001"/>
+    </geometry>
+  </collision>
+</link>
+<link name="knee-bend-motor-bracket-hip_1">
+  <inertial>
+    <origin xyz="-0.0038111444447288256 -0.01598260549680081 -0.008478998621304334" rpy="0 0 0"/>
+    <mass value="0.0107277558839088"/>
+    <inertia ixx="1.93139707619719e-06" iyy="6.52187217630501e-07" izz="2.10236783725592e-06" ixy="-4.64701319342865e-07" iyz="-7.37049479173783e-09" ixz="2.26759346512173e-08"/>
+  </inertial>
+  <visual>
+    <origin xyz="-0.053 -0.0 -0.012" rpy="0 0 0"/>
+    <geometry>
+      <mesh filename="package://humanoidrightleg_description/meshes/knee-bend-motor-bracket-hip_1.stl" scale="0.001 0.001 0.001"/>
+    </geometry>
+    <material name="opaque191191191"/>
+  </visual>
+  <collision>
+    <origin xyz="-0.053 -0.0 -0.012" rpy="0 0 0"/>
+    <geometry>
+      <mesh filename="package://humanoidrightleg_description/meshes/knee-bend-motor-bracket-hip_1.stl" scale="0.001 0.001 0.001"/>
+    </geometry>
+  </collision>
+</link>
+<link name="knee-bend-motor-bracket-hip__1__1">
+  <inertial>
+    <origin xyz="-0.0038110401177033695 -0.015982284411230948 0.00847899862130437" rpy="0 0 0"/>
+    <mass value="0.0107277558839088"/>
+    <inertia ixx="1.93139815764031e-06" iyy="6.52186136187552e-07" izz="2.10236783725603e-06" ixy="-4.64699830864174e-07" iyz="7.36572442646488e-09" ixz="-2.26774846368458e-08"/>
+  </inertial>
+  <visual>
+    <origin xyz="-0.053 -0.0 -0.071" rpy="0 0 0"/>
+    <geometry>
+      <mesh filename="package://humanoidrightleg_description/meshes/knee-bend-motor-bracket-hip__1__1.stl" scale="0.001 0.001 0.001"/>
+    </geometry>
+    <material name="opaque191191191"/>
+  </visual>
+  <collision>
+    <origin xyz="-0.053 -0.0 -0.071" rpy="0 0 0"/>
+    <geometry>
+      <mesh filename="package://humanoidrightleg_description/meshes/knee-bend-motor-bracket-hip__1__1.stl" scale="0.001 0.001 0.001"/>
+    </geometry>
+  </collision>
+</link>
+<link name="RMD-X10-S2_MIR4Stator_1">
+  <inertial>
+    <origin xyz="0.01637821078173142 -0.04960639092028741 0.02917930007753167" rpy="0 0 0"/>
+    <mass value="1.55306904844426"/>
+    <inertia ixx="0.00285644715024275" iyy="0.00292757747778099" izz="0.00369780684183896" ixy="-7.224770955105431e-11" iyz="-1.67010427996753e-05" ixz="4.91373074174017e-10"/>
+  </inertial>
+  <visual>
+    <origin xyz="0.088088 0.048294 -0.012" rpy="0 0 0"/>
+    <geometry>
+      <mesh filename="package://humanoidrightleg_description/meshes/RMD-X10-S2_MIR4Stator_1.stl" scale="0.001 0.001 0.001"/>
+    </geometry>
+    <material name="opaque727161"/>
+  </visual>
+  <collision>
+    <origin xyz="0.088088 0.048294 -0.012" rpy="0 0 0"/>
+    <geometry>
+      <mesh filename="package://humanoidrightleg_description/meshes/RMD-X10-S2_MIR4Stator_1.stl" scale="0.001 0.001 0.001"/>
+    </geometry>
+  </collision>
+</link>
+<link name="RMD-X10-S2_MIR4Rotor_1">
+  <inertial>
+    <origin xyz="-2.1161672708047696e-06 1.6410298648822375e-05 -0.011165974681643147" rpy="0 0 0"/>
+    <mass value="0.236112274637419"/>
+    <inertia ixx="5.68531155036552e-05" iyy="5.7336639638052e-05" izz="7.49151450519106e-05" ixy="-6.93161398973574e-08" iyz="-2.3024874127751e-08" ixz="3.23928483927753e-09"/>
+  </inertial>
+  <visual>
+    <origin xyz="0.07171 0.0987 -0.073" rpy="0 0 0"/>
+    <geometry>
+      <mesh filename="package://humanoidrightleg_description/meshes/RMD-X10-S2_MIR4Rotor_1.stl" scale="0.001 0.001 0.001"/>
+    </geometry>
+    <material name="opaque727161"/>
+  </visual>
+  <collision>
+    <origin xyz="0.07171 0.0987 -0.073" rpy="0 0 0"/>
+    <geometry>
+      <mesh filename="package://humanoidrightleg_description/meshes/RMD-X10-S2_MIR4Rotor_1.stl" scale="0.001 0.001 0.001"/>
+    </geometry>
+  </collision>
+</link>
+<link name="thigh-outer-encoder-mount__1__1">
+  <inertial>
+    <origin xyz="0.012347854634024116 0.013208765079570972 0.032156691836600845" rpy="0 0 0"/>
+    <mass value="0.0298095431336914"/>
+    <inertia ixx="1.94825595458806e-05" iyy="2.41201920848334e-05" izz="1.15362961084242e-05" ixy="1.68477718283047e-06" iyz="2.74493604757647e-06" ixz="-8.44793203533018e-06"/>
+  </inertial>
+  <visual>
+    <origin xyz="0.12471 0.0987 -0.071" rpy="0 0 0"/>
+    <geometry>
+      <mesh filename="package://humanoidrightleg_description/meshes/thigh-outer-encoder-mount__1__1.stl" scale="0.001 0.001 0.001"/>
+    </geometry>
+    <material name="opaque191191191"/>
+  </visual>
+  <collision>
+    <origin xyz="0.12471 0.0987 -0.071" rpy="0 0 0"/>
+    <geometry>
+      <mesh filename="package://humanoidrightleg_description/meshes/thigh-outer-encoder-mount__1__1.stl" scale="0.001 0.001 0.001"/>
+    </geometry>
+  </collision>
+</link>
+<link name="limit-bracket-knee_1">
+  <inertial>
+    <origin xyz="0.038087477180112975 0.00807344983971442 0.00200543257018429" rpy="0 0 0"/>
+    <mass value="0.0111496094135345"/>
+    <inertia ixx="2.38308173316804e-06" iyy="7.30358139373011e-06" izz="9.59027505735826e-06" ixy="-3.43104983657425e-06" iyz="-2.22510402278926e-08" ixz="9.00308746571408e-09"/>
+  </inertial>
+  <visual>
+    <origin xyz="0.088088 0.149106 -0.071" rpy="0 0 0"/>
+    <geometry>
+      <mesh filename="package://humanoidrightleg_description/meshes/limit-bracket-knee_1.stl" scale="0.001 0.001 0.001"/>
+    </geometry>
+    <material name="opaque191191191"/>
+  </visual>
+  <collision>
+    <origin xyz="0.088088 0.149106 -0.071" rpy="0 0 0"/>
+    <geometry>
+      <mesh filename="package://humanoidrightleg_description/meshes/limit-bracket-knee_1.stl" scale="0.001 0.001 0.001"/>
+    </geometry>
+  </collision>
+</link>
+<link name="hip-motor-bracket-v5-right_MIR__1__1">
+  <inertial>
+    <origin xyz="0.02831909901748353 -0.047580037015949136 0.004499999933483212" rpy="0 0 0"/>
+    <mass value="0.0629963904640038"/>
+    <inertia ixx="4.19044662888547e-05" iyy="6.28781864330074e-05" izz="0.000103932201450599" ixy="3.22752392715876e-05" iyz="-3.294155855211589e-14" ixz="-8.834716270188225e-14"/>
+  </inertial>
+  <visual>
+    <origin xyz="0.064174 0.00177 -0.071" rpy="0 0 0"/>
+    <geometry>
+      <mesh filename="package://humanoidrightleg_description/meshes/hip-motor-bracket-v5-right_MIR__1__1.stl" scale="0.001 0.001 0.001"/>
+    </geometry>
+    <material name="opaque245245245"/>
+  </visual>
+  <collision>
+    <origin xyz="0.064174 0.00177 -0.071" rpy="0 0 0"/>
+    <geometry>
+      <mesh filename="package://humanoidrightleg_description/meshes/hip-motor-bracket-v5-right_MIR__1__1.stl" scale="0.001 0.001 0.001"/>
+    </geometry>
+  </collision>
+</link>
+<link name="NO-NC_Bump_Switch__1__1">
+  <inertial>
+    <origin xyz="0.0006098597083060778 -0.005605907200915444 0.0033312733839520187" rpy="0 0 0"/>
+    <mass value="0.00155039406540348"/>
+    <inertia ixx="7.02105776941548e-08" iyy="4.0851523004421e-08" izz="6.23354983706727e-08" ixy="-2.17632942777091e-08" iyz="-6.72541221178337e-09" ixz="-3.57596510481949e-09"/>
+  </inertial>
+  <visual>
+    <origin xyz="0.011323 0.125712 -0.06881" rpy="0 0 0"/>
+    <geometry>
+      <mesh filename="package://humanoidrightleg_description/meshes/NO-NC_Bump_Switch__1__1.stl" scale="0.001 0.001 0.001"/>
+    </geometry>
+    <material name="opaque252525"/>
+  </visual>
+  <collision>
+    <origin xyz="0.011323 0.125712 -0.06881" rpy="0 0 0"/>
+    <geometry>
+      <mesh filename="package://humanoidrightleg_description/meshes/NO-NC_Bump_Switch__1__1.stl" scale="0.001 0.001 0.001"/>
+    </geometry>
+  </collision>
+</link>
+<link name="NO-NC_Bump_Switch_1">
+  <inertial>
+    <origin xyz="0.004177517614909906 -0.003788104538661019 0.003331273383956626" rpy="0 0 0"/>
+    <mass value="0.00155039406540348"/>
+    <inertia ixx="3.02967040915035e-08" iyy="8.07653966070994e-08" izz="6.23354983707032e-08" ixy="7.23583235206848e-09" iyz="-1.06008157257925e-09" ixz="7.54287232483715e-09"/>
+  </inertial>
+  <visual>
+    <origin xyz="0.085847 0.163362 -0.06881" rpy="0 0 0"/>
+    <geometry>
+      <mesh filename="package://humanoidrightleg_description/meshes/NO-NC_Bump_Switch_1.stl" scale="0.001 0.001 0.001"/>
+    </geometry>
+    <material name="opaque252525"/>
+  </visual>
+  <collision>
+    <origin xyz="0.085847 0.163362 -0.06881" rpy="0 0 0"/>
+    <geometry>
+      <mesh filename="package://humanoidrightleg_description/meshes/NO-NC_Bump_Switch_1.stl" scale="0.001 0.001 0.001"/>
+    </geometry>
+  </collision>
+</link>
+<link name="hip-ex-al-base_MIR_1">
+  <inertial>
+    <origin xyz="-9.949334274853006e-06 0.00014878773576262883 0.013372003753055584" rpy="0 0 0"/>
+    <mass value="0.145590268667055"/>
+    <inertia ixx="7.31142837610502e-05" iyy="8.03439498425385e-05" izz="0.000138206755307654" ixy="-4.95170279436914e-07" iyz="-1.74096248714692e-06" ixz="1.18687228429994e-07"/>
+  </inertial>
+  <visual>
+    <origin xyz="0.07171 0.0987 -0.073" rpy="0 0 0"/>
+    <geometry>
+      <mesh filename="package://humanoidrightleg_description/meshes/hip-ex-al-base_MIR_1.stl" scale="0.001 0.001 0.001"/>
+    </geometry>
+    <material name="opaque22122113"/>
+  </visual>
+  <collision>
+    <origin xyz="0.07171 0.0987 -0.073" rpy="0 0 0"/>
+    <geometry>
+      <mesh filename="package://humanoidrightleg_description/meshes/hip-ex-al-base_MIR_1.stl" scale="0.001 0.001 0.001"/>
+    </geometry>
+  </collision>
+</link>
+<link name="motorcap-KNEE_MIR_1">
+  <inertial>
+    <origin xyz="-0.00010458296907729647 0.001536971231776929 0.010431913725907738" rpy="0 0 0"/>
+    <mass value="0.10890019522501"/>
+    <inertia ixx="5.28935639643557e-05" iyy="5.74293989570557e-05" izz="0.000103470968365381" ixy="-3.10665335403418e-07" iyz="9.03944422473183e-07" ixz="-6.16246300980637e-08"/>
+  </inertial>
+  <visual>
+    <origin xyz="0.07171 0.0987 -0.1" rpy="0 0 0"/>
+    <geometry>
+      <mesh filename="package://humanoidrightleg_description/meshes/motorcap-KNEE_MIR_1.stl" scale="0.001 0.001 0.001"/>
+    </geometry>
+    <material name="opaque22122113"/>
+  </visual>
+  <collision>
+    <origin xyz="0.07171 0.0987 -0.1" rpy="0 0 0"/>
+    <geometry>
+      <mesh filename="package://humanoidrightleg_description/meshes/motorcap-KNEE_MIR_1.stl" scale="0.001 0.001 0.001"/>
+    </geometry>
+  </collision>
+</link>
+<link name="2020_300mm__1__1">
+  <inertial>
+    <origin xyz="0.0002251870068053774 -0.15033302956237268 -0.00999999999999844" rpy="0 0 0"/>
+    <mass value="0.158693154300952"/>
+    <inertia ixx="0.00119118913093242" iyy="1.84090653089298e-05" izz="0.0011966651702521" ixy="8.03254427837138e-05" iyz="1.734723475976807e-17" ixz="1.517883041479706e-18"/>
+  </inertial>
+  <visual>
+    <origin xyz="0.063093 0.078066 -0.11" rpy="0 0 0"/>
+    <geometry>
+      <mesh filename="package://humanoidrightleg_description/meshes/2020_300mm__1__1.stl" scale="0.001 0.001 0.001"/>
+    </geometry>
+    <material name="opaque727161"/>
+  </visual>
+  <collision>
+    <origin xyz="0.063093 0.078066 -0.11" rpy="0 0 0"/>
+    <geometry>
+      <mesh filename="package://humanoidrightleg_description/meshes/2020_300mm__1__1.stl" scale="0.001 0.001 0.001"/>
+    </geometry>
+  </collision>
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
File: humanoidrightleg_description/urdf/materials.xacro (robot description, xacro)
@@ -28,9 +28,9 @@
   <color rgba="0.5137254901960784 0.4235294117647059 0.37254901960784315 1.0"/>
 </material>
-<material name="opaque2550255">
-  <color rgba="1.0 0.0 1.0 1.0"/>
-</material>
 <material name="powder_coat_green">
   <color rgba="0.26666666666666666 0.5882352941176471 0.2823529411764706 0.0"/>
 </material>
+<material name="steel_satin">
+  <color rgba="0.6274509803921569 0.6274509803921569 0.6274509803921569 1.0"/>
+</material>
 </robot>
