Commit message: Implement code changes to enhance functionality and improve performance

File: hyperspawn_dropbear_description/urdf/arm.xacro (robot description, xacro)
@@ -6,1770 +6,1782 @@
     Find - xyz="(.+)\s(.+)\s(.+)" r
     Replace - xyz="$1 $2 ${sign*$3}" r
+    Find
+      <inertia\s+ixx="([^"]+)"\s+iyy="([^"]+)"\s+izz="([^"]+)"\s+ixy="([^"]+)"\s+iyz="([^"]+)"\s+ixz="([^"]+)"\s*/>
+    Replace
+      <inertia ixx="$1" iyy="$2" izz="$3" ixy="${sign*$4}" iyz="${sign*$5}" ixz="$6"/>
+      hyperspawn_dropbear_description/meshes/${folder}
+      link name="${prefix}_
+      joint name="${prefix}_${prefix}_
    -->
+    <!-- <link name="${prefix}_base_link">
+      <inertial>
+        <origin xyz="-6.496817022290221e-15 0 ${sign*0.005}" rpy="0 0 0"/>
+        <mass value="0.49623462441733"/>
+        <inertia ixx="0.000272043421613551" iyy="0.000272043421603598" izz="0.000535816266143527" ixy="${sign*-8.924416761146857e-20}" iyz="${sign*0}" ixz="3.081487911019577e-33"/>
+      </inertial>
+      <visual>
+        <origin xyz="0 0 ${sign*0}" rpy="0 0 0"/>
+        <geometry>
+          <mesh filename="package://hyperspawn_dropbear_description/meshes/${folder}/base_link.stl" scale="0.001 0.001 0.001"/>
+        </geometry>
+        <material name="steel_satin"/>
+      </visual>
+      <collision>
+        <origin xyz="0 0 ${sign*0}" rpy="0 0 0"/>
+        <geometry>
+          <mesh filename="package://hyperspawn_dropbear_description/meshes/${folder}/base_link.stl" scale="0.001 0.001 0.001"/>
+        </geometry>
+      </collision>
+    </link> -->
     <xacro:macro name="arm_macro" params="prefix folder parent sign *origin">
-        <!-- <link name="${prefix}_base_link">
-          <inertial>
-            <origin xyz="-4.564684959507811e-14 -1.297744842251468e-14 ${sign*-0.00040000000000051}" rpy="0 0 0"/>
-            <mass value="0.0710251267123582"/>
-            <inertia ixx="1.03755872605632e-05" iyy="1.03755872605639e-05" izz="2.04552364931589e-05" ixy="2.231104194494098e-20" iyz="-3.993969333038147e-17" ixz="8.809863505376990e-17"/>
-          </inertial>
-          <visual>
-            <origin xyz="0 0 ${sign*0}" rpy="0 0 0"/>
-            <geometry>
-              <mesh filename="package://hyperspawn_dropbear_description/meshes/${folder}/base_link.stl" scale="0.001 0.001 0.001"/>
-            </geometry>
-            <material name="opaque2550255"/>
-          </visual>
-          <collision>
-            <origin xyz="0 0 ${sign*0}" rpy="0 0 0"/>
-            <geometry>
-              <mesh filename="package://hyperspawn_dropbear_description/meshes/${folder}/base_link.stl" scale="0.001 0.001 0.001"/>
-            </geometry>
-          </collision>
-        </link> -->
-        <link name="${prefix}_2020_100mm__9__1">
-          <inertial>
-            <origin xyz="1.4980442800229068e-14 5.199887469533773e-15 ${sign*0.049999999999999795}" rpy="0 0 0"/>
-            <mass value="0.019591747444562"/>
-            <inertia ixx="1.71247911414457e-05" iyy="1.71247911416276e-05" izz="1.59666987542057e-06" ixy="-6.394884621840706e-17" iyz="2.518172085831656e-18" ixz="7.829445091340370e-18"/>
-          </inertial>
-          <visual>
-            <origin xyz="0.0 0.0 ${sign*-0.0021}" rpy="0 0 0"/>
-            <geometry>
-              <mesh filename="package://hyperspawn_dropbear_description/meshes/${folder}/2020_100mm__9__1.stl" scale="0.001 0.001 0.001"/>
-            </geometry>
-            <material name="opaque727161"/>
-          </visual>
-          <collision>
-            <origin xyz="0.0 0.0 ${sign*-0.0021}" rpy="0 0 0"/>
-            <geometry>
-              <mesh filename="package://hyperspawn_dropbear_description/meshes/${folder}/2020_100mm__9__1.stl" scale="0.001 0.001 0.001"/>
-            </geometry>
-          </collision>
-        </link>
-        <link name="${prefix}_shoulder-roll-al-mot_MIR1__1__1">
-          <inertial>
-            <origin xyz="0.005127204279605231 -0.01578027268886943 ${sign*0.013349013943228552}" rpy="0 0 0"/>
-            <mass value="0.0139822805624322"/>
-            <inertia ixx="1.33357850186962e-06" iyy="2.39192509601408e-06" izz="1.95321408998418e-06" ixy="-3.84446207640792e-07" iyz="1.4147058742276e-08" ixz="-4.62978754176702e-09"/>
-          </inertial>
-          <visual>
-            <origin xyz="0.0 -0.0 ${sign*-0.0021}" rpy="0 0 0"/>
-            <geometry>
-              <mesh filename="package://hyperspawn_dropbear_description/meshes/${folder}/shoulder-roll-al-mot_MIR1__1__1.stl" scale="0.001 0.001 0.001"/>
-            </geometry>
-            <material name="opaque245245245"/>
-          </visual>
-          <collision>
-            <origin xyz="0.0 -0.0 ${sign*-0.0021}" rpy="0 0 0"/>
-            <geometry>
-              <mesh filename="package://hyperspawn_dropbear_description/meshes/${folder}/shoulder-roll-al-mot_MIR1__1__1.stl" scale="0.001 0.001 0.001"/>
-            </geometry>
-          </collision>
-        </link>
-        <link name="${prefix}_shoulder-roll-al-mot_MIR1__2__1">
-          <inertial>
-            <origin xyz="-0.005127204279607458 0.015780272688869185 ${sign*0.013349013943228556}" rpy="0 0 0"/>
-            <mass value="0.0139822805624322"/>
-            <inertia ixx="1.33357850186963e-06" iyy="2.39192509601406e-06" izz="1.95321408998418e-06" ixy="-3.84446207640812e-07" iyz="-1.41470587422785e-08" ixz="4.62978754176003e-09"/>
-          </inertial>
-          <visual>
-            <origin xyz="0.0 -0.0 ${sign*-0.0021}" rpy="0 0 0"/>
-            <geometry>
-              <mesh filename="package://hyperspawn_dropbear_description/meshes/${folder}/shoulder-roll-al-mot_MIR1__2__1.stl" scale="0.001 0.001 0.001"/>
-            </geometry>
-            <material name="opaque245245245"/>
-          </visual>
-          <collision>
-            <origin xyz="0.0 -0.0 ${sign*-0.0021}" rpy="0 0 0"/>
-            <geometry>
-              <mesh filename="package://hyperspawn_dropbear_description/meshes/${folder}/shoulder-roll-al-mot_MIR1__2__1.stl" scale="0.001 0.001 0.001"/>
-            </geometry>
-          </collision>
-        </link>
-        <link name="${prefix}_yaw-cap_1">
-          <inertial>
-            <origin xyz="-8.404754804490673e-15 2.1068804545096473e-14 ${sign*-0.006586829858195878}" rpy="0 0 0"/>
-            <mass value="0.0147970811486"/>
-            <inertia ixx="2.47144498176233e-06" iyy="4.12036554274002e-06" izz="2.86340658923296e-06" ixy="-5.99005456426396e-07" iyz="2.946851009227335e-18" ixz="-1.059818412580698e-18"/>
-          </inertial>
-          <visual>
-            <origin xyz="0.0 0.0 ${sign*-0.1021}" rpy="0 0 0"/>
-            <geometry>
-              <mesh filename="package://hyperspawn_dropbear_description/meshes/${folder}/yaw-cap_1.stl" scale="0.001 0.001 0.001"/>
-            </geometry>
-            <material name="opaque245245245"/>
-          </visual>
-          <collision>
-            <origin xyz="0.0 0.0 ${sign*-0.1021}" rpy="0 0 0"/>
-            <geometry>
-              <mesh filename="package://hyperspawn_dropbear_description/meshes/${folder}/yaw-cap_1.stl" scale="0.001 0.001 0.001"/>
-            </geometry>
-          </collision>
-        </link>
-        <link name="${prefix}_yaw-waist-adapter-motor-exal_MIR1_1">
-          <inertial>
-            <origin xyz="-0.0022354396247523025 0.006879975731446575 ${sign*0.049999999999987436}" rpy="0 0 0"/>
-            <mass value="0.0374132377219994"/>
-            <inertia ixx="7.74698902279246e-06" iyy="1.35806331978027e-05" izz="1.28983762196582e-05" ixy="-2.11919529319787e-06" iyz="-1.897353801849633e-19" ixz="3.642241673193491e-20"/>
-          </inertial>
-          <visual>
-            <origin xyz="0.0 -0.0 ${sign*-0.0021}" rpy="0 0 0"/>
-            <geometry>
-              <mesh filename="package://hyperspawn_dropbear_description/meshes/${folder}/yaw-waist-adapter-motor-exal_MIR1_1.stl" scale="0.001 0.001 0.001"/>
-            </geometry>
-            <material name="opaque245245245"/>
-          </visual>
-          <collision>
-            <origin xyz="0.0 -0.0 ${sign*-0.0021}" rpy="0 0 0"/>
-            <geometry>
-              <mesh filename="package://hyperspawn_dropbear_description/meshes/${folder}/yaw-waist-adapter-motor-exal_MIR1_1.stl" scale="0.001 0.001 0.001"/>
-            </geometry>
-          </collision>
-        </link>
-        <link name="${prefix}_front-bearing-adapter-shoulder_1">
-          <inertial>
-            <origin xyz="0.012476625956564928 0.01204671407588206 ${sign*-0.00900000000002072}" rpy="0 0 0"/>
-            <mass value="0.023683107739144"/>
-            <inertia ixx="3.64971689005244e-06" iyy="7.09787565227239e-06" izz="5.22213010024979e-06" ixy="-1.2526169920336e-06" iyz="9.893344823930228e-19" ixz="-3.184843881676169e-19"/>
-          </inertial>
-          <visual>
-            <origin xyz="0.021006 -0.014204 ${sign*-0.0611}" rpy="0 0 0"/>
-            <geometry>
-              <mesh filename="package://hyperspawn_dropbear_description/meshes/${folder}/front-bearing-adapter-shoulder_1.stl" scale="0.001 0.001 0.001"/>
-            </geometry>
-            <material name="opaque191191191"/>
-          </visual>
-          <collision>
-            <origin xyz="0.021006 -0.014204 ${sign*-0.0611}" rpy="0 0 0"/>
-            <geometry>
-              <mesh filename="package://hyperspawn_dropbear_description/meshes/${folder}/front-bearing-adapter-shoulder_1.stl" scale="0.001 0.001 0.001"/>
-            </geometry>
-          </collision>
-        </link>
-        <link name="${prefix}_shoulder-ex-al-interface__2__1">
-          <inertial>
-            <origin xyz="0.01738138579865837 -0.0030497886170603797 ${sign*-0.008999999999991598}" rpy="0 0 0"/>
-            <mass value="0.027893677646265"/>
-            <inertia ixx="4.32482586114369e-06" iyy="8.39411157893946e-06" izz="6.30628010967354e-06" ixy="-1.47825456629198e-06" iyz="2.466898755583424e-17" ixz="7.404253805128741e-17"/>
-          </inertial>
-          <visual>
-            <origin xyz="0.011735 0.014328 ${sign*-0.0611}" rpy="0 0 0"/>
-            <geometry>
-              <mesh filename="package://hyperspawn_dropbear_description/meshes/${folder}/shoulder-ex-al-interface__2__1.stl" scale="0.001 0.001 0.001"/>
-            </geometry>
-            <material name="opaque22122113"/>
-          </visual>
-          <collision>
-            <origin xyz="0.011735 0.014328 ${sign*-0.0611}" rpy="0 0 0"/>
-            <geometry>
-              <mesh filename="package://hyperspawn_dropbear_description/meshes/${folder}/shoulder-ex-al-interface__2__1.stl" scale="0.001 0.001 0.001"/>
-            </geometry>
-          </collision>
-        </link>
-        <link name="${prefix}_RMD-X8-Pro_MIR8_MIR1__1__1">
-          <inertial>
-            <origin xyz="0.0067650965649745445 -0.020808521702550438 ${sign*0.00046176070349858434}" rpy="0 0 0"/>
-            <mass value="0.0658409996798309"/>
-            <inertia ixx="6.73245559130172e-05" iyy="9.09727241934292e-05" izz="6.35281702686579e-05" ixy="-8.59564716294938e-06" iyz="7.14503501851588e-07" ixz="-2.30317369534993e-07"/>
-          </inertial>
-          <visual>
-            <origin xyz="-0.008343 0.025679 ${sign*-0.0521}" rpy="0 0 0"/>
-            <geometry>
-              <mesh filename="package://hyperspawn_dropbear_description/meshes/${folder}/RMD-X8-Pro_MIR8_MIR1__1__1.stl" scale="0.001 0.001 0.001"/>
-            </geometry>
-            <material name="opaque13110895"/>
-          </visual>
-          <collision>
-            <origin xyz="-0.008343 0.025679 ${sign*-0.0521}" rpy="0 0 0"/>
-            <geometry>
-              <mesh filename="package://hyperspawn_dropbear_description/meshes/${folder}/RMD-X8-Pro_MIR8_MIR1__1__1.stl" scale="0.001 0.001 0.001"/>
-            </geometry>
-          </collision>
-        </link>
-        <link name="${prefix}_shoulder-motor-bicep-rotor-bracket_1">
-          <inertial>
-            <origin xyz="0.011585383104448774 -0.002019144805998477 ${sign*0.006894585665480131}" rpy="0 0 0"/>
-            <mass value="0.0242631871440445"/>
-            <inertia ixx="7.32924174579478e-06" iyy="1.01897271688699e-05" izz="4.02506203897297e-06" ixy="-1.03913215530172e-06" iyz="-4.23772294446241e-07" ixz="-1.30423701412823e-06"/>
-          </inertial>
-          <visual>
-            <origin xyz="-0.059876 0.048364 ${sign*-0.0521}" rpy="0 0 0"/>
-            <geometry>
-              <mesh filename="package://hyperspawn_dropbear_description/meshes/${folder}/shoulder-motor-bicep-rotor-bracket_1.stl" scale="0.001 0.001 0.001"/>
-            </geometry>
-            <material name="opaque245245245"/>
-          </visual>
-          <collision>
-            <origin xyz="-0.059876 0.048364 ${sign*-0.0521}" rpy="0 0 0"/>
-            <geometry>
-              <mesh filename="package://hyperspawn_dropbear_description/meshes/${folder}/shoulder-motor-bicep-rotor-bracket_1.stl" scale="0.001 0.001 0.001"/>
-            </geometry>
-          </collision>
-        </link>
-        <link name="${prefix}_bicep-rear-motor-adapter_1">
-          <inertial>
-            <origin xyz="-0.0018929355342764131 0.016127672677199507 ${sign*0.015500000000001603}" rpy="0 0 0"/>
-            <mass value="0.0281681226709944"/>
-            <inertia ixx="6.66789269228993e-06" iyy="5.24554656234814e-06" izz="6.37785740381877e-06" ixy="1.31824458087614e-06" iyz="1.694065894508601e-19" ixz="-5.421010862427522e-20"/>
-          </inertial>
-          <visual>
-            <origin xyz="-0.076995 0.042802 ${sign*-0.0506}" rpy="0 0 0"/>
-            <geometry>
-              <mesh filename="package://hyperspawn_dropbear_description/meshes/${folder}/bicep-rear-motor-adapter_1.stl" scale="0.001 0.001 0.001"/>
-            </geometry>
-            <material name="opaque191191191"/>
-          </visual>
-          <collision>
-            <origin xyz="-0.076995 0.042802 ${sign*-0.0506}" rpy="0 0 0"/>
-            <geometry>
-              <mesh filename="package://hyperspawn_dropbear_description/meshes/${folder}/bicep-rear-motor-adapter_1.stl" scale="0.001 0.001 0.001"/>
-            </geometry>
-          </collision>
-        </link>
-        <link name="${prefix}_bicep-shoulder-bracket-exal__1__1">
-          <inertial>
-            <origin xyz="0.011983042446585573 -0.004518260205938709 ${sign*0.005535150009386286}" rpy="0 0 0"/>
-            <mass value="0.0119000299936683"/>
-            <inertia ixx="1.06039831340363e-06" iyy="1.52523000194053e-06" izz="2.34706806988364e-06" ixy="-1.688599950433e-07" iyz="6.776263578034403e-21" ixz="1.355252715606881e-20"/>
-          </inertial>
-          <visual>
-            <origin xyz="-0.065252 0.006662 ${sign*-0.0761}" rpy="0 0 0"/>
-            <geometry>
-              <mesh filename="package://hyperspawn_dropbear_description/meshes/${folder}/bicep-shoulder-bracket-exal__1__1.stl" scale="0.001 0.001 0.001"/>
-            </geometry>
-            <material name="opaque245245245"/>
-          </visual>
-          <collision>
-            <origin xyz="-0.065252 0.006662 ${sign*-0.0761}" rpy="0 0 0"/>
-            <geometry>
-              <mesh filename="package://hyperspawn_dropbear_description/meshes/${folder}/bicep-shoulder-bracket-exal__1__1.stl" scale="0.001 0.001 0.001"/>
-            </geometry>
-          </collision>
-        </link>
-        <link name="${prefix}_bicep-shoulder-bracket-exal__2__1">
-          <inertial>
-            <origin xyz="0.011983042446582756 -0.004518260205939313 ${sign*-0.0054648499906134115}" rpy="0 0 0"/>
-            <mass value="0.0119000299936683"/>
-            <inertia ixx="1.06039831340363e-06" iyy="1.5252300019405e-06" izz="2.34706806988363e-06" ixy="-1.68859995043294e-07" iyz="6.776263578034403e-21" ixz="1.355252715606881e-20"/>
-          </inertial>
-          <visual>
-            <origin xyz="-0.065252 0.006662 ${sign*-0.0561}" rpy="0 0 0"/>
-            <geometry>
-              <mesh filename="package://hyperspawn_dropbear_description/meshes/${folder}/bicep-shoulder-bracket-exal__2__1.stl" scale="0.001 0.001 0.001"/>
-            </geometry>
-            <material name="opaque245245245"/>
-          </visual>
-          <collision>
-            <origin xyz="-0.065252 0.006662 ${sign*-0.0561}" rpy="0 0 0"/>
-            <geometry>
-              <mesh filename="package://hyperspawn_dropbear_description/meshes/${folder}/bicep-shoulder-bracket-exal__2__1.stl" scale="0.001 0.001 0.001"/>
-            </geometry>
-          </collision>
-        </link>
-        <link name="${prefix}_2020_100mm__8__1">
-          <inertial>
-            <origin xyz="-0.02187147869637933 0.034952359549973555 ${sign*-0.009999999999981746}" rpy="0 0 0"/>
-            <mass value="0.019591747444562"/>
-            <inertia ixx="1.5641987506042e-05" iyy="3.0794735109847e-06" izz="1.71247911413717e-05" ixy="4.56360033803824e-06" iyz="-7.738493006115288e-18" ixz="2.507217523872729e-18"/>
-          </inertial>
-          <visual>
-            <origin xyz="-0.097956 0.010231 ${sign*-0.0761}" rpy="0 0 0"/>
-            <geometry>
-              <mesh filename="package://hyperspawn_dropbear_description/meshes/${folder}/2020_100mm__8__1.stl" scale="0.001 0.001 0.001"/>
-            </geometry>
-            <material name="opaque727161"/>
-          </visual>
-          <collision>
-            <origin xyz="-0.097956 0.010231 ${sign*-0.0761}" rpy="0 0 0"/>
-            <geometry>
-              <mesh filename="package://hyperspawn_dropbear_description/meshes/${folder}/2020_100mm__8__1.stl" scale="0.001 0.001 0.001"/>
-            </geometry>
-          </collision>
-        </link>
-        <link name="${prefix}_yaw-waist-adapter-motor-exal_MIR1__5__1">
-          <inertial>
-            <origin xyz="0.008570545572160838 -0.049788080074744674 ${sign*1.457167719820518e-15}" rpy="0 0 0"/>
-            <mass value="0.0374132377219994"/>
-            <inertia ixx="1.41382993236902e-05" iyy="1.30292783846948e-05" izz="7.05842073186832e-06" ixy="4.02875438314004e-07" iyz="-6.776263578034403e-21" ixz="5.421010862427522e-20"/>
-          </inertial>
-          <visual>
-            <origin xyz="-0.060634 -0.072274 ${sign*-0.0661}" rpy="0 0 0"/>
-            <geometry>
-              <mesh filename="package://hyperspawn_dropbear_description/meshes/${folder}/yaw-waist-adapter-motor-exal_MIR1__5__1.stl" scale="0.001 0.001 0.001"/>
-            </geometry>
-            <material name="opaque245245245"/>
-          </visual>
-          <collision>
-            <origin xyz="-0.060634 -0.072274 ${sign*-0.0661}" rpy="0 0 0"/>
-            <geometry>
-              <mesh filename="package://hyperspawn_dropbear_description/meshes/${folder}/yaw-waist-adapter-motor-exal_MIR1__5__1.stl" scale="0.001 0.001 0.001"/>
-            </geometry>
-          </collision>
-        </link>
-        <link name="${prefix}_bicep-shoulder-bracket-exal_1">
-          <inertial>
-            <origin xyz="-0.014231130165287431 -0.020921360581575885 ${sign*-0.007214849990613441}" rpy="0 0 0"/>
-            <mass value="0.0119000299936683"/>
-            <inertia ixx="1.06039831340366e-06" iyy="1.5252300019405e-06" izz="2.34706806988368e-06" ixy="-1.68859995043294e-07" iyz="6.776263578034403e-21" ixz="1.355252715606881e-20"/>
-          </inertial>
-          <visual>
-            <origin xyz="-0.070144 -0.075364 ${sign*-0.05785}" rpy="0 0 0"/>
-            <geometry>
-              <mesh filename="package://hyperspawn_dropbear_description/meshes/${folder}/bicep-shoulder-bracket-exal_1.stl" scale="0.001 0.001 0.001"/>
-            </geometry>
-            <material name="opaque245245245"/>
-          </visual>
-          <collision>
-            <origin xyz="-0.070144 -0.075364 ${sign*-0.05785}" rpy="0 0 0"/>
-            <geometry>
-              <mesh filename="package://hyperspawn_dropbear_description/meshes/${folder}/bicep-shoulder-bracket-exal_1.stl" scale="0.001 0.001 0.001"/>
-            </geometry>
-          </collision>
-        </link>
-        <link name="${prefix}_shoulder-front_1">
-          <inertial>
-            <origin xyz="-0.007463364992977992 -0.010559925065031256 ${sign*0.010000000000000855}" rpy="0 0 0"/>
-            <mass value="0.0285901454621081"/>
-            <inertia ixx="5.24738535853905e-06" iyy="5.75381404316444e-06" izz="5.10534101569437e-06" ixy="-1.12882167821954e-07" iyz="-4.118613002729310e-17" ixz="-1.249543003789544e-16"/>
-          </inertial>
-          <visual>
-            <origin xyz="-0.04393 -0.058961 ${sign*-0.0561}" rpy="0 0 0"/>
-            <geometry>
-              <mesh filename="package://hyperspawn_dropbear_description/meshes/${folder}/shoulder-front_1.stl" scale="0.001 0.001 0.001"/>
-            </geometry>
-            <material name="opaque191191191"/>
-          </visual>
-          <collision>
-            <origin xyz="-0.04393 -0.058961 ${sign*-0.0561}" rpy="0 0 0"/>
-            <geometry>
-              <mesh filename="package://hyperspawn_dropbear_description/meshes/${folder}/shoulder-front_1.stl" scale="0.001 0.001 0.001"/>
-            </geometry>
-          </collision>
-        </link>
-        <link name="${prefix}_bicep-shoulder-bracket-exal__3__1">
-          <inertial>
-            <origin xyz="0.011982869834713333 -0.00451836058157562 ${sign*0.0055351500093866746}" rpy="0 0 0"/>
-            <mass value="0.0119000299936683"/>
-            <inertia ixx="1.06039831340366e-06" iyy="1.52523000194053e-06" izz="2.3470680698837e-06" ixy="-1.688599950433e-07" iyz="6.776263578034403e-21" ixz="1.355252715606881e-20"/>
-          </inertial>
-          <visual>
-            <origin xyz="-0.04393 -0.058961 ${sign*-0.0761}" rpy="0 0 0"/>
-            <geometry>
-              <mesh filename="package://hyperspawn_dropbear_description/meshes/${folder}/bicep-shoulder-bracket-exal__3__1.stl" scale="0.001 0.001 0.001"/>
-            </geometry>
-            <material name="opaque245245245"/>
-          </visual>
-          <collision>
-            <origin xyz="-0.04393 -0.058961 ${sign*-0.0761}" rpy="0 0 0"/>
-            <geometry>
-              <mesh filename="package://hyperspawn_dropbear_description/meshes/${folder}/bicep-shoulder-bracket-exal__3__1.stl" scale="0.001 0.001 0.001"/>
-            </geometry>
-          </collision>
-        </link>
-        <link name="${prefix}_shoulder-cap_1">
-          <inertial>
-            <origin xyz="-0.034857061179216664 -0.006155365677712535 ${sign*-0.02572256391671531}" rpy="0 0 0"/>
-            <mass value="0.046227678179176"/>
-            <inertia ixx="1.76465028282704e-05" iyy="3.51734867524788e-05" izz="2.25355319862365e-05" ixy="-6.39975511036637e-06" iyz="-1.32005071311637e-06" ixz="-4.02230543927391e-06"/>
-          </inertial>
-          <visual>
-            <origin xyz="-0.024494 -0.060532 ${sign*-0.0811}" rpy="0 0 0"/>
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