Commit message: Comment out dynamics parameters in arm_.xacro joints for clarity

File: hyperspawn_dropbear_description/urdf/arm_.xacro (robot description, xacro)
@@ -1740,8 +1740,8 @@
                 <velocity>10.0</velocity>
               </limit>
-              <dynamics>
+              <!-- <dynamics>
                 <damping>10.0</damping>
                 <friction>0.50</friction>
-              </dynamics>
+              </dynamics> -->
             </joint>
             <joint name="${prefix}_Revolute47_gz" type="revolute">
@@ -1757,8 +1757,8 @@
                 <upper>${PI}</upper>
               </limit>
-              <dynamics>
+              <!-- <dynamics>
                 <damping>1.0</damping>
                 <friction>0.5</friction>
-              </dynamics>
+              </dynamics> -->
             </joint>
             <joint name="${prefix}_Recolute48_gz" type="revolute">
@@ -1773,8 +1773,8 @@
                 <upper>${PI}</upper>
               </limit>
-              <dynamics>
+              <!-- <dynamics>
                 <damping>2.0</damping>
                 <friction>0.10</friction>
-              </dynamics>
+              </dynamics> -->
             </joint>
           </gazebo>
