Commit message: Uncomment leg and battery macros in URDF, adjust base link origin for improved positioning

File: hyperspawn_dropbear_description/urdf/hyperspawn_dropbear.urdf.xacro (robot description, xacro)
@@ -14,7 +14,7 @@
     <xacro:include filename="$(find hyperspawn_dropbear_description)/urdf/arm.xacro"/>
     <!-- Leg Xacro -->
-    <!-- <xacro:include filename="$(find hyperspawn_dropbear_description)/urdf/leg.xacro"/> -->
+    <xacro:include filename="$(find hyperspawn_dropbear_description)/urdf/leg.xacro"/>
     <!-- Battery xacro -->
-    <!-- <xacro:include filename="$(find hyperspawn_dropbear_description)/urdf/battery.xacro"/> -->
+    <xacro:include filename="$(find hyperspawn_dropbear_description)/urdf/battery.xacro"/>
     <!-- ros2 control -->
     <!-- <xacro:include filename="$(find hyperspawn_dropbear_description)/urdf/ros2_control/hyperspawn_dropbear_description.ros2_control.xacro"/> -->
@@ -26,5 +26,5 @@
     <!-- base_link to world joint -->
     <joint name="base_link_sim_world_joint" type="fixed">
-        <origin xyz="0.0 0.0 0.5" rpy="${PI/2} 0.0 0.0"/>
+        <origin xyz="0.0 0.0 1.5" rpy="${PI/2} 0.0 0.0"/>
         <!-- <origin xyz="0.0 0.0 1.4" rpy="${0} 0.0 0.0"/> -->
         <parent link="world"/>
@@ -62,7 +62,7 @@
     </xacro:arm_macro> -->
     <!-- Right Leg -->
-    <!-- <xacro:leg_macro prefix = "RL" folder = "rightleg" parent = "PG_motor-yaw-cap_1" sign = "1">
-        <origin xyz="0 0 0" rpy="${5/9 * PI} 0 0"/>
-    </xacro:leg_macro> -->
+    <xacro:leg_macro prefix = "RL" folder = "right_leg" parent = "PG_motor-yaw-cap_1" sign = "1">
+        <origin xyz="0 0 0" rpy="${1/18 * PI} 0 0"/>
+    </xacro:leg_macro>
     <!-- <xacro:leg_macro prefix = "RL" folder = "rightleg" parent = "RL_base_link" sign = "1">
         <origin xyz="0 0 0" rpy="${5/9 * PI} 0 0"/>
@@ -76,6 +76,6 @@
     </xacro:leg_macro> -->
     <!-- Battery -->
-     <!-- <xacro:battery_macro parent = "torso_left-battery-mount_1">
+     <xacro:battery_macro parent = "torso_left-battery-mount_1">
         <origin xyz="0.08 -0.028115 0.03632" rpy="0 0 0"/>
-     </xacro:battery_macro> -->
+     </xacro:battery_macro>
 </robot>

Commit message: Add gazebo plugin for ROS control and update arm macros for consistency

File: hyperspawn_dropbear_description/urdf/hyperspawn_dropbear.urdf.xacro (robot description, xacro)
@@ -19,4 +19,9 @@
     <!-- ros2 control -->
     <!-- <xacro:include filename="$(find hyperspawn_dropbear_description)/urdf/ros2_control/hyperspawn_dropbear_description.ros2_control.xacro"/> -->
+    <gazebo>
+        <plugin filename="libgazebo_ros_control.so" name="gazebo_ros_control">
+          <robotNamespace>/</robotNamespace>
+        </plugin>
+      </gazebo>
     <!-- World Link -->
     <link name="world"/>
@@ -40,7 +45,7 @@
     </joint> -->
     <!-- Head -->
-    <xacro:head_macro prefix="head" parent = "torso_base_link">
+    <!-- <xacro:head_macro prefix="head" parent = "torso_base_link">
         <origin xyz="0.0985 0.0798 0.069747" rpy="0 ${PI/2} 0"/>
-    </xacro:head_macro>
+    </xacro:head_macro> -->
     <!-- waist -->
     <xacro:pelvicgirdle_macro prefix="PG" parent = "torso_lumbar-strap_1">
@@ -49,5 +54,6 @@
     <!-- Right Arm-->
     <xacro:arm_macro prefix="RH" folder = "right_arm" parent = "torso_RMD-X10Rotot_1" sign = "1">
-        <origin xyz="0.0 0.0 0.0" rpy="0 0 ${-7*PI/12}"/>
+        <!-- <origin xyz="0.0 0.0 0.0" rpy="0 0 ${-7*PI/12}"/> -->
+        <origin xyz="0.0 0.0 0.0" rpy="0 0 0"/>
     </xacro:arm_macro>
     <!-- <xacro:arm_macro prefix="RH" folder = "rightarm" parent = "RH_base_link" sign = "1">
@@ -55,20 +61,20 @@
     </xacro:arm_macro> -->
     <!-- Left Arm -->
-    <!-- <xacro:arm_macro prefix="LH" folder = "leftarm" parent = "torso_RMD-X10__1_Rotor_1" sign = "-1">
+    <xacro:arm_macro prefix="LH" folder = "left_arm" parent = "torso_RMD-X10__1_Rotor_1" sign = "-1">
         <origin xyz="0.0 0.0 0.0" rpy="0 0 0"/>
-    </xacro:arm_macro> -->
+    </xacro:arm_macro>
     <!-- <xacro:arm_macro prefix="LH" folder = "leftarm" parent = "LH_base_link" sign = "-1">
         <origin xyz="0.0 0.0 0.0" rpy="0 0 0"/>
     </xacro:arm_macro> -->
     <!-- Right Leg -->
-    <xacro:leg_macro prefix = "RL" folder = "right_leg" parent = "PG_motor-yaw-cap_1" sign = "1">
+    <!-- <xacro:leg_macro prefix = "RL" folder = "right_leg" parent = "PG_motor-yaw-cap_1" sign = "1">
         <origin xyz="0 0 0" rpy="${1/18 * PI} 0 0"/>
-    </xacro:leg_macro>
+    </xacro:leg_macro> -->
     <!-- <xacro:leg_macro prefix = "RL" folder = "rightleg" parent = "RL_base_link" sign = "1">
         <origin xyz="0 0 0" rpy="${5/9 * PI} 0 0"/>
     </xacro:leg_macro> -->
     <!-- Left Leg -->
-    <!-- <xacro:leg_macro prefix = "LL" folder = "leftleg" parent = "PG_motor-yaw-cap__1__1" sign = "-1">
-        <origin xyz="0 0 0" rpy="${4/9 * PI} 0 0"/>
+    <!-- <xacro:leg_macro prefix = "LL" folder = "left_leg" parent = "PG_motor-yaw-cap__1__1" sign = "-1">
+        <origin xyz="0 0 0" rpy="${-1/18 * PI} 0 0"/>
     </xacro:leg_macro> -->
     <!-- <xacro:leg_macro prefix = "LL" folder = "leftleg" parent = "RL_base_link" sign = "-1">
@@ -76,6 +82,6 @@
     </xacro:leg_macro> -->
     <!-- Battery -->
-     <xacro:battery_macro parent = "torso_left-battery-mount_1">
+     <!-- <xacro:battery_macro parent = "torso_left-battery-mount_1">
         <origin xyz="0.08 -0.028115 0.03632" rpy="0 0 0"/>
-     </xacro:battery_macro>
+     </xacro:battery_macro> -->
 </robot>

Commit message: Rename world link to sim_world and uncomment relevant macros for clarity

File: hyperspawn_dropbear_description/urdf/hyperspawn_dropbear.urdf.xacro (robot description, xacro)
@@ -25,5 +25,5 @@
       </gazebo>
     <!-- World Link -->
-    <link name="world"/>
+    <link name="sim_world"/>
     <!-- Torso macro -->
      <xacro:torso_macro prefix="torso">
@@ -33,5 +33,5 @@
         <origin xyz="0.0 0.0 1.5" rpy="${PI/2} 0.0 0.0"/>
         <!-- <origin xyz="0.0 0.0 1.4" rpy="${0} 0.0 0.0"/> -->
-        <parent link="world"/>
+        <parent link="sim_world"/>
         <!-- Torso Base link -->
         <child link="torso_base_link"/>
@@ -45,7 +45,7 @@
     </joint> -->
     <!-- Head -->
-    <!-- <xacro:head_macro prefix="head" parent = "torso_base_link">
+    <xacro:head_macro prefix="head" parent = "torso_base_link">
         <origin xyz="0.0985 0.0798 0.069747" rpy="0 ${PI/2} 0"/>
-    </xacro:head_macro> -->
+    </xacro:head_macro>
     <!-- waist -->
     <xacro:pelvicgirdle_macro prefix="PG" parent = "torso_lumbar-strap_1">
@@ -68,20 +68,20 @@
     </xacro:arm_macro> -->
     <!-- Right Leg -->
-    <!-- <xacro:leg_macro prefix = "RL" folder = "right_leg" parent = "PG_motor-yaw-cap_1" sign = "1">
+    <xacro:leg_macro prefix = "RL" folder = "right_leg" parent = "PG_motor-yaw-cap_1" sign = "1">
         <origin xyz="0 0 0" rpy="${1/18 * PI} 0 0"/>
-    </xacro:leg_macro> -->
+    </xacro:leg_macro>
     <!-- <xacro:leg_macro prefix = "RL" folder = "rightleg" parent = "RL_base_link" sign = "1">
         <origin xyz="0 0 0" rpy="${5/9 * PI} 0 0"/>
     </xacro:leg_macro> -->
     <!-- Left Leg -->
-    <!-- <xacro:leg_macro prefix = "LL" folder = "left_leg" parent = "PG_motor-yaw-cap__1__1" sign = "-1">
+    <xacro:leg_macro prefix = "LL" folder = "left_leg" parent = "PG_motor-yaw-cap__1__1" sign = "-1">
         <origin xyz="0 0 0" rpy="${-1/18 * PI} 0 0"/>
-    </xacro:leg_macro> -->
+    </xacro:leg_macro>
     <!-- <xacro:leg_macro prefix = "LL" folder = "leftleg" parent = "RL_base_link" sign = "-1">
         <origin xyz="0.0 0.2 0.0" rpy="${4/9 * PI} 0 0"/>
     </xacro:leg_macro> -->
     <!-- Battery -->
-     <!-- <xacro:battery_macro parent = "torso_left-battery-mount_1">
+     <xacro:battery_macro parent = "torso_left-battery-mount_1">
         <origin xyz="0.08 -0.028115 0.03632" rpy="0 0 0"/>
-     </xacro:battery_macro> -->
+     </xacro:battery_macro>
 </robot>

Commit message: Fix ros2_control include path and adjust joint origin for sim_world link

File: hyperspawn_dropbear_description/urdf/hyperspawn_dropbear.urdf.xacro (robot description, xacro)
@@ -18,10 +18,5 @@
     <xacro:include filename="$(find hyperspawn_dropbear_description)/urdf/battery.xacro"/>
     <!-- ros2 control -->
-    <!-- <xacro:include filename="$(find hyperspawn_dropbear_description)/urdf/ros2_control/hyperspawn_dropbear_description.ros2_control.xacro"/> -->
-    <gazebo>
-        <plugin filename="libgazebo_ros_control.so" name="gazebo_ros_control">
-          <robotNamespace>/</robotNamespace>
-        </plugin>
-      </gazebo>
+    <xacro:include filename="$(find hyperspawn_dropbear_description)/urdf/ros2_control/hyperspawn_dropbear.ros2_control.xacro"/>
     <!-- World Link -->
     <link name="sim_world"/>
@@ -31,5 +26,5 @@
     <!-- base_link to world joint -->
     <joint name="base_link_sim_world_joint" type="fixed">
-        <origin xyz="0.0 0.0 1.5" rpy="${PI/2} 0.0 0.0"/>
+        <origin xyz="0.0 0.0 1.4" rpy="${PI/2} 0.0 0.0"/>
         <!-- <origin xyz="0.0 0.0 1.4" rpy="${0} 0.0 0.0"/> -->
         <parent link="sim_world"/>

Commit message: Comment out unused xacro macros and adjust joint origin parameters for clarity

File: hyperspawn_dropbear_description/urdf/hyperspawn_dropbear.urdf.xacro (robot description, xacro)
@@ -22,14 +22,14 @@
     <link name="sim_world"/>
     <!-- Torso macro -->
-     <xacro:torso_macro prefix="torso">
-     </xacro:torso_macro>
+     <!-- <xacro:torso_macro prefix="torso">
+     </xacro:torso_macro> -->
     <!-- base_link to world joint -->
     <joint name="base_link_sim_world_joint" type="fixed">
-        <origin xyz="0.0 0.0 1.4" rpy="${PI/2} 0.0 0.0"/>
-        <!-- <origin xyz="0.0 0.0 1.4" rpy="${0} 0.0 0.0"/> -->
+        <!-- <origin xyz="0.0 0.0 1.4" rpy="${PI/2} 0.0 0.0"/> -->
+        <origin xyz="0.0 0.0 1.4" rpy="${5/9 * PI} 0.0 0.0"/>
         <parent link="sim_world"/>
         <!-- Torso Base link -->
-        <child link="torso_base_link"/>
-        <!-- <child link="RL_base_link"/> -->
+        <!-- <child link="torso_base_link"/> -->
+        <child link="RL_base_link"/>
         <!-- <child link="RH_base_link"/> -->
     </joint>
@@ -40,33 +40,32 @@
     </joint> -->
     <!-- Head -->
-    <xacro:head_macro prefix="head" parent = "torso_base_link">
+    <!-- <xacro:head_macro prefix="head" parent = "torso_base_link">
         <origin xyz="0.0985 0.0798 0.069747" rpy="0 ${PI/2} 0"/>
-    </xacro:head_macro>
+    </xacro:head_macro> -->
     <!-- waist -->
-    <xacro:pelvicgirdle_macro prefix="PG" parent = "torso_lumbar-strap_1">
+    <!-- <xacro:pelvicgirdle_macro prefix="PG" parent = "torso_lumbar-strap_1">
         <origin xyz="-0.023253 -0.021955 0.0" rpy="0 0 0"/>
-    </xacro:pelvicgirdle_macro>
+    </xacro:pelvicgirdle_macro> -->
     <!-- Right Arm-->
-    <xacro:arm_macro prefix="RH" folder = "right_arm" parent = "torso_RMD-X10Rotot_1" sign = "1">
-        <!-- <origin xyz="0.0 0.0 0.0" rpy="0 0 ${-7*PI/12}"/> -->
+    <!-- <xacro:arm_macro prefix="RH" folder = "right_arm" parent = "torso_RMD-X10Rotot_1" sign = "1">
         <origin xyz="0.0 0.0 0.0" rpy="0 0 0"/>
-    </xacro:arm_macro>
+    </xacro:arm_macro> -->
     <!-- <xacro:arm_macro prefix="RH" folder = "rightarm" parent = "RH_base_link" sign = "1">
         <origin xyz="0.0 0.0 0.0" rpy="0 0 0"/>
     </xacro:arm_macro> -->
     <!-- Left Arm -->
-    <xacro:arm_macro prefix="LH" folder = "left_arm" parent = "torso_RMD-X10__1_Rotor_1" sign = "-1">
+    <!-- <xacro:arm_macro prefix="LH" folder = "left_arm" parent = "torso_RMD-X10__1_Rotor_1" sign = "-1">
         <origin xyz="0.0 0.0 0.0" rpy="0 0 0"/>
-    </xacro:arm_macro>
+    </xacro:arm_macro> -->
     <!-- <xacro:arm_macro prefix="LH" folder = "leftarm" parent = "LH_base_link" sign = "-1">
         <origin xyz="0.0 0.0 0.0" rpy="0 0 0"/>
     </xacro:arm_macro> -->
     <!-- Right Leg -->
-    <xacro:leg_macro prefix = "RL" folder = "right_leg" parent = "PG_motor-yaw-cap_1" sign = "1">
+    <!-- <xacro:leg_macro prefix = "RL" folder = "right_leg" parent = "PG_motor-yaw-cap_1" sign = "1">
         <origin xyz="0 0 0" rpy="${1/18 * PI} 0 0"/>
+    </xacro:leg_macro> -->
+    <xacro:leg_macro prefix = "RL" folder = "right_leg" parent = "RL_base_link" sign = "1">
+        <origin xyz="0 0 0.01" rpy="0 0 0"/>
     </xacro:leg_macro>
-    <!-- <xacro:leg_macro prefix = "RL" folder = "rightleg" parent = "RL_base_link" sign = "1">
-        <origin xyz="0 0 0" rpy="${5/9 * PI} 0 0"/>
-    </xacro:leg_macro> -->
     <!-- Left Leg -->
     <!-- <xacro:leg_macro prefix = "LL" folder = "left_leg" parent = "PG_motor-yaw-cap__1__1" sign = "-1">
@@ -77,6 +76,6 @@
     </xacro:leg_macro> -->
     <!-- Battery -->
-     <xacro:battery_macro parent = "torso_left-battery-mount_1">
+     <!-- <xacro:battery_macro parent = "torso_left-battery-mount_1">
         <origin xyz="0.08 -0.028115 0.03632" rpy="0 0 0"/>
-     </xacro:battery_macro>
+     </xacro:battery_macro> -->
 </robot>

Commit message: Uncomment torso macro and adjust joint parameters for improved robot structure

File: hyperspawn_dropbear_description/urdf/hyperspawn_dropbear.urdf.xacro (robot description, xacro)
@@ -22,14 +22,14 @@
     <link name="sim_world"/>
     <!-- Torso macro -->
-     <!-- <xacro:torso_macro prefix="torso">
-     </xacro:torso_macro> -->
+     <xacro:torso_macro prefix="torso">
+     </xacro:torso_macro>
     <!-- base_link to world joint -->
     <joint name="base_link_sim_world_joint" type="fixed">
-        <!-- <origin xyz="0.0 0.0 1.4" rpy="${PI/2} 0.0 0.0"/> -->
-        <origin xyz="0.0 0.0 1.4" rpy="${5/9 * PI} 0.0 0.0"/>
+        <origin xyz="0.0 0.0 1.4" rpy="${PI/2} 0.0 0.0"/>
+        <!-- <origin xyz="0.0 0.0 1.4" rpy="${5/9 * PI} 0.0 0.0"/> -->
         <parent link="sim_world"/>
         <!-- Torso Base link -->
-        <!-- <child link="torso_base_link"/> -->
-        <child link="RL_base_link"/>
+        <child link="torso_base_link"/>
+        <!-- <child link="RL_base_link"/> -->
         <!-- <child link="RH_base_link"/> -->
     </joint>
@@ -40,42 +40,42 @@
     </joint> -->
     <!-- Head -->
-    <!-- <xacro:head_macro prefix="head" parent = "torso_base_link">
+    <xacro:head_macro prefix="head" parent = "torso_base_link">
         <origin xyz="0.0985 0.0798 0.069747" rpy="0 ${PI/2} 0"/>
-    </xacro:head_macro> -->
+    </xacro:head_macro>
     <!-- waist -->
-    <!-- <xacro:pelvicgirdle_macro prefix="PG" parent = "torso_lumbar-strap_1">
+    <xacro:pelvicgirdle_macro prefix="PG" parent = "torso_lumbar-strap_1">
         <origin xyz="-0.023253 -0.021955 0.0" rpy="0 0 0"/>
-    </xacro:pelvicgirdle_macro> -->
+    </xacro:pelvicgirdle_macro>
     <!-- Right Arm-->
-    <!-- <xacro:arm_macro prefix="RH" folder = "right_arm" parent = "torso_RMD-X10Rotot_1" sign = "1">
+    <xacro:arm_macro prefix="RH" folder = "right_arm" parent = "torso_RMD-X10Rotot_1" sign = "1">
         <origin xyz="0.0 0.0 0.0" rpy="0 0 0"/>
-    </xacro:arm_macro> -->
+    </xacro:arm_macro>
     <!-- <xacro:arm_macro prefix="RH" folder = "rightarm" parent = "RH_base_link" sign = "1">
         <origin xyz="0.0 0.0 0.0" rpy="0 0 0"/>
     </xacro:arm_macro> -->
     <!-- Left Arm -->
-    <!-- <xacro:arm_macro prefix="LH" folder = "left_arm" parent = "torso_RMD-X10__1_Rotor_1" sign = "-1">
+    <xacro:arm_macro prefix="LH" folder = "left_arm" parent = "torso_RMD-X10__1_Rotor_1" sign = "-1">
         <origin xyz="0.0 0.0 0.0" rpy="0 0 0"/>
-    </xacro:arm_macro> -->
+    </xacro:arm_macro>
     <!-- <xacro:arm_macro prefix="LH" folder = "leftarm" parent = "LH_base_link" sign = "-1">
         <origin xyz="0.0 0.0 0.0" rpy="0 0 0"/>
     </xacro:arm_macro> -->
     <!-- Right Leg -->
-    <!-- <xacro:leg_macro prefix = "RL" folder = "right_leg" parent = "PG_motor-yaw-cap_1" sign = "1">
+    <xacro:leg_macro prefix = "RL" folder = "right_leg" parent = "PG_motor-yaw-cap_1" sign = "1">
         <origin xyz="0 0 0" rpy="${1/18 * PI} 0 0"/>
+    </xacro:leg_macro>
+    <!-- <xacro:leg_macro prefix = "RL" folder = "right_leg" parent = "RL_base_link" sign = "1">
+        <origin xyz="0 0 0.01" rpy="0 0 0"/>
     </xacro:leg_macro> -->
-    <xacro:leg_macro prefix = "RL" folder = "right_leg" parent = "RL_base_link" sign = "1">
-        <origin xyz="0 0 0.01" rpy="0 0 0"/>
+    <!-- Left Leg -->
+    <xacro:leg_macro prefix = "LL" folder = "left_leg" parent = "PG_motor-yaw-cap__1__1" sign = "-1">
+        <origin xyz="0 0 0" rpy="${-1/18 * PI} 0 0"/>
     </xacro:leg_macro>
-    <!-- Left Leg -->
-    <!-- <xacro:leg_macro prefix = "LL" folder = "left_leg" parent = "PG_motor-yaw-cap__1__1" sign = "-1">
-        <origin xyz="0 0 0" rpy="${-1/18 * PI} 0 0"/>
-    </xacro:leg_macro> -->
     <!-- <xacro:leg_macro prefix = "LL" folder = "leftleg" parent = "RL_base_link" sign = "-1">
         <origin xyz="0.0 0.2 0.0" rpy="${4/9 * PI} 0 0"/>
     </xacro:leg_macro> -->
     <!-- Battery -->
-     <!-- <xacro:battery_macro parent = "torso_left-battery-mount_1">
+     <xacro:battery_macro parent = "torso_left-battery-mount_1">
         <origin xyz="0.08 -0.028115 0.03632" rpy="0 0 0"/>
-     </xacro:battery_macro> -->
+     </xacro:battery_macro>
 </robot>

Commit message: Fix link name in URDF: change 'sim_world' to 'world' for consistency

File: hyperspawn_dropbear_description/urdf/hyperspawn_dropbear.urdf.xacro (robot description, xacro)
@@ -20,5 +20,5 @@
     <xacro:include filename="$(find hyperspawn_dropbear_description)/urdf/ros2_control/hyperspawn_dropbear.ros2_control.xacro"/>
     <!-- World Link -->
-    <link name="sim_world"/>
+    <link name="world"/>
     <!-- Torso macro -->
      <xacro:torso_macro prefix="torso">
@@ -28,5 +28,5 @@
         <origin xyz="0.0 0.0 1.4" rpy="${PI/2} 0.0 0.0"/>
         <!-- <origin xyz="0.0 0.0 1.4" rpy="${5/9 * PI} 0.0 0.0"/> -->
-        <parent link="sim_world"/>
+        <parent link="world"/>
         <!-- Torso Base link -->
         <child link="torso_base_link"/>
