Commit message: Comment out dynamics parameters in leg.xacro joints for clarity

File: hyperspawn_dropbear_description/urdf/leg.xacro (robot description, xacro)
@@ -2850,8 +2850,8 @@
               <velocity>10.0</velocity>
           </limit>
-          <dynamics>
+          <!-- <dynamics>
               <damping>10.0</damping>
               <friction>0.1</friction>
-          </dynamics>
+          </dynamics> -->
       </joint>
     <joint name="${prefix}_Revolute72gz" type="revolute">
@@ -2868,8 +2868,8 @@
             <velocity>10.0</velocity>
         </limit>
-        <dynamics>
+        <!-- <dynamics>
             <damping>10.0</damping>
             <friction>0.1</friction>
-        </dynamics>
+        </dynamics> -->
     </joint>
     <joint name="${prefix}_Revolute73gz" type="revolute">
@@ -2886,8 +2886,8 @@
             <velocity>10.0</velocity>
         </limit>
-        <dynamics>
+        <!-- <dynamics>
             <damping>10.0</damping>
             <friction>0.1</friction>
-        </dynamics>
+        </dynamics> -->
     </joint>
     <joint name="${prefix}_Revolute113gz" type="revolute">
@@ -2904,8 +2904,8 @@
             <velocity>10.0</velocity>
         </limit>
-        <dynamics>
+        <!-- <dynamics>
             <damping>10.0</damping>
             <friction>0.10</friction>
-        </dynamics>
+        </dynamics> -->
     </joint>
     <joint name="${prefix}_Revolute114gz" type="revolute">
@@ -2922,8 +2922,8 @@
             <velocity>10.0</velocity>
         </limit>
-        <dynamics>
+        <!-- <dynamics>
             <damping>0.0</damping>
             <friction>0.0</friction>
-        </dynamics>
+        </dynamics> -->
     </joint>
 </gazebo>

Commit message: Refactor leg.xacro: uncomment base link and change joint types to continuous for improved clarity and functionality

File: hyperspawn_dropbear_description/urdf/leg.xacro (robot description, xacro)
@@ -2,5 +2,5 @@
 <robot name="humanoidrightleg" xmlns:xacro="http://www.ros.org/wiki/xacro">
   <xacro:macro name="leg_macro" params="prefix folder parent sign *origin">
-<!-- <link name="${prefix}_base_link">
+<link name="${prefix}_base_link">
   <inertial>
     <origin xyz="-2.137404171899072e-14 0 ${sign*0.005}" rpy="0 0 0"/>
@@ -21,5 +21,5 @@
     </geometry>
   </collision>
-</link> -->
+</link>
 <link name="${prefix}_RMD-X10-S2_MIR4__3_Stator_1">
   <inertial>
@@ -2232,5 +2232,5 @@
   <child link="${prefix}_RMD-X10-S2_MIR4__3_Stator_1"/>
   <axis xyz="0.0 0.0 -1.0"/>
-  <limit upper="${PI}" lower="${-PI}" velocity="10.0" effort="100.0"/>
+  <limit upper="${PI}" lower="${-PI}" velocity="10.0" effort="10.0"/>
 </joint>
 <joint name="${prefix}_Rigid 3" type="fixed">
@@ -2284,5 +2284,5 @@
   <child link="${prefix}_RMD-X10-S2_MIR4Rotor_1"/>
   <axis xyz="0.0 0.0 1.0"/>
-  <limit upper="${PI}" lower="${-PI}" velocity="10.0" effort="100.0"/>>
+  <limit upper="${PI}" lower="${-PI}" velocity="10.0" effort="100.0"/>
 </joint>
 <joint name="${prefix}_Rigid 14" type="fixed">
@@ -2356,17 +2356,15 @@
   <child link="${prefix}_bearingstrap__1__1"/>
 </joint>
-<joint name="${prefix}_Revolute28" type="revolute">
+<joint name="${prefix}_Revolute28" type="continuous">
   <origin xyz="0.001021 -0.014965 ${sign*-0.01}" rpy="0 0 0"/>
   <parent link="${prefix}_bearingstrap__1__1"/>
   <child link="${prefix}_skateboard-bearing__13__1"/>
   <axis xyz="0.0 0.0 -1.0"/>
-  <limit upper="${PI}" lower="${-PI}" velocity="10.0" effort="100.0"/>
-</joint>
-<joint name="${prefix}_Revolute29" type="revolute">
+</joint>
+<joint name="${prefix}_Revolute29" type="continuous">
   <origin xyz="0.001021 -0.014965 ${sign*0.01}" rpy="0 0 0"/>
   <parent link="${prefix}_bearingstrap__1__1"/>
   <child link="${prefix}_skateboard-bearing__14__1"/>
   <axis xyz="0.0 0.0 1.0"/>
-  <limit upper="${PI}" lower="${-PI}" velocity="10.0" effort="100.0"/>
 </joint>
 <joint name="${prefix}_Rigid 30" type="fixed">
@@ -2385,17 +2383,15 @@
   <child link="${prefix}_skateboard-bearing__15__1"/>
 </joint>
-<joint name="${prefix}_Revolute33" type="revolute">
+<joint name="${prefix}_Revolute33" type="continuous">
   <origin xyz="0.0 0.0 ${sign*0.0005}" rpy="0 0 0"/>
   <parent link="${prefix}_skateboard-bearing__15__1"/>
   <child link="${prefix}_bearingstrap_1"/>
   <axis xyz="0.0 0.0 -1.0"/>
-  <limit upper="${PI}" lower="${-PI}" velocity="10.0" effort="100.0"/>
-</joint>
-<joint name="${prefix}_Revolute34" type="revolute">
+</joint>
+<joint name="${prefix}_Revolute34" type="continuous">
   <origin xyz="0.0 0.0 ${sign*0.02}" rpy="0 0 0"/>
   <parent link="${prefix}_bearingstrap_1"/>
   <child link="${prefix}_skateboard-bearing_1"/>
   <axis xyz="0.0 0.0 1.0"/>
-  <limit upper="${PI}" lower="${-PI}" velocity="10.0" effort="100.0"/>
 </joint>
 <joint name="${prefix}_Rigid 35" type="fixed">
@@ -2409,17 +2405,15 @@
   <child link="${prefix}_skateboard-bearing__8__1"/>
 </joint>
-<joint name="${prefix}_Revolute37" type="revolute">
+<joint name="${prefix}_Revolute37" type="continuous">
   <origin xyz="0.0 0.0 ${sign*0.000335}" rpy="0 0 0"/>
   <parent link="${prefix}_skateboard-bearing__8__1"/>
   <child link="${prefix}_bearingstrap-inner-thigh_1"/>
   <axis xyz="0.0 0.0 1.0"/>
-  <limit upper="${PI}" lower="${-PI}" velocity="10.0" effort="100.0"/>
-</joint>
-<joint name="${prefix}_Revolute38" type="revolute">
+</joint>
+<joint name="${prefix}_Revolute38" type="continuous">
   <origin xyz="0.0 0.0 ${sign*-0.02}" rpy="0 0 0"/>
   <parent link="${prefix}_bearingstrap-inner-thigh_1"/>
   <child link="${prefix}_skateboard-bearing__9__1"/>
   <axis xyz="0.0 0.0 -1.0"/>
-  <limit upper="${PI}" lower="${-PI}" velocity="10.0" effort="100.0"/>
 </joint>
 <joint name="${prefix}_Rigid 40" type="fixed">
@@ -2453,31 +2447,27 @@
   <child link="${prefix}_double-bracket_1"/>
 </joint>
-<joint name="${prefix}_Revolute46" type="revolute">
+<joint name="${prefix}_Revolute46" type="continuous">
   <origin xyz="-0.000105 -0.015 ${sign*0.01}" rpy="0 0 0"/>
   <parent link="${prefix}_double-bracket_1"/>
   <child link="${prefix}_skateboard-bearing__11__1"/>
   <axis xyz="0.0 0.0 1.0"/>
-  <limit upper="${PI}" lower="${-PI}" velocity="10.0" effort="100.0"/>
-</joint>
-<joint name="${prefix}_Revolute47" type="revolute">
+</joint>
+<joint name="${prefix}_Revolute47" type="continuous">
   <origin xyz="-0.060103 -0.014581 ${sign*0.01}" rpy="0 0 0"/>
   <parent link="${prefix}_double-bracket_1"/>
   <child link="${prefix}_skateboard-bearing__20__1"/>
   <axis xyz="0.0 0.0 1.0"/>
-  <limit upper="${PI}" lower="${-PI}" velocity="10.0" effort="100.0"/>
-</joint>
-<joint name="${prefix}_Revolute48" type="revolute">
+</joint>
+<joint name="${prefix}_Revolute48" type="continuous">
   <origin xyz="-0.000105 -0.015 ${sign*-0.01}" rpy="0 0 0"/>
   <parent link="${prefix}_double-bracket_1"/>
   <child link="${prefix}_skateboard-bearing__10__1"/>
   <axis xyz="0.0 0.0 -1.0"/>
-  <limit upper="${PI}" lower="${-PI}" velocity="10.0" effort="100.0"/>
-</joint>
-<joint name="${prefix}_Revolute49" type="revolute">
+</joint>
+<joint name="${prefix}_Revolute49" type="continuous">
   <origin xyz="-0.060103 -0.014581 ${sign*-0.01}" rpy="0 0 0"/>
   <parent link="${prefix}_double-bracket_1"/>
   <child link="${prefix}_skateboard-bearing__16__1"/>
   <axis xyz="0.0 0.0 -1.0"/>
-  <limit upper="${PI}" lower="${-PI}" velocity="10.0" effort="100.0"/>
 </joint>
 <!-- <joint name="${prefix}_Rigid 50" type="fixed">
@@ -2516,10 +2506,9 @@
   <child link="${prefix}_skateboard-bearing__12__1"/>
 </joint>
-<joint name="${prefix}_Revolute57" type="revolute">
+<joint name="${prefix}_Revolute57" type="continuous">
   <origin xyz="0.0 0.0 ${sign*0.0}" rpy="0 0 0"/>
   <parent link="${prefix}_skateboard-bearing__19__1"/>
   <child link="${prefix}_double-bracket-10deg_MIR_MIR_MIR_1"/>
   <axis xyz="0.0 0.0 1.0"/>
-  <limit upper="${PI}" lower="${-PI}" velocity="10.0" effort="100.0"/>
 </joint>
 <joint name="${prefix}_Rigid 58" type="fixed">
@@ -2610,10 +2599,9 @@
   <child link="${prefix}_motor-calf-exal-mount_2"/>
 </joint>
-<joint name="${prefix}_Revolute81" type="revolute">
+<joint name="${prefix}_Revolute81" type="continuous">
   <origin xyz="-0.023945 -0.033572 ${sign*0.008354}" rpy="0 0 0"/>
   <parent link="${prefix}_RMD-X8-Pro_MIR8_MIR1_1"/>
   <child link="${prefix}_calf-motor-driver-ext_2"/>
   <axis xyz="-0.004243 0.173596 0.984808"/>
-  <limit upper="${PI}" lower="${-PI}" velocity="10.0" effort="100.0"/>
 </joint>
 <joint name="${prefix}_Rigid 82" type="fixed">
@@ -2642,10 +2630,9 @@
   <child link="${prefix}_ankle-side-bracket_1"/>
 </joint>
-<joint name="${prefix}_Revolute87" type="revolute">
+<joint name="${prefix}_Revolute87" type="continuous">
   <origin xyz="0.000885 -0.036193 ${sign*-0.003771}" rpy="0 0 0"/>
   <parent link="${prefix}_ankle-thick_1"/>
   <child link="${prefix}_basis_left_1"/>
   <axis xyz="0.004243 -0.173596 -0.984808"/>
-  <limit upper="${PI}" lower="${-PI}" velocity="10.0" effort="100.0"/>
 </joint>
 <joint name="${prefix}_Revolute88" type="revolute">
@@ -2656,10 +2643,9 @@
   <limit upper="${PI}" lower="${-PI}" velocity="10.0" effort="100.0"/>
 </joint>
-<joint name="${prefix}_Revolute89" type="revolute">
+<joint name="${prefix}_Revolute89" type="continuous">
   <origin xyz="-0.01765 -0.038762 ${sign*0.016911}" rpy="0 0 0"/>
   <parent link="${prefix}_basis_left_1"/>
   <child link="${prefix}_skateboard-bearing_left_1"/>
   <axis xyz="-0.998253 -0.058776 0.00606"/>
-  <limit upper="${PI}" lower="${-PI}" velocity="10.0" effort="100.0"/>
 </joint>
 <joint name="${prefix}_Rigid 90" type="fixed">
@@ -2763,17 +2749,15 @@
   <child link="${prefix}_ankle-motor-driver-bracket_left_1"/>
 </joint>
-<joint name="${prefix}_Revolute111" type="revolute">
+<joint name="${prefix}_Revolute111" type="continuous">
   <origin xyz="0.039873 0.005664 ${sign*0.026589}" rpy="0 0 0"/>
   <parent link="${prefix}_calf-motor-driver-ext_2"/>
   <child link="${prefix}_210mm-tie-rod_v1_1"/>
   <axis xyz="-0.004243 0.173596 0.984808"/>
-  <limit upper="${PI}" lower="${-PI}" velocity="10.0" effort="100.0"/>
-</joint>
-<joint name="${prefix}_Revolute112" type="revolute">
+</joint>
+<joint name="${prefix}_Revolute112" type="continuous">
   <origin xyz="0.036763 -0.020444 ${sign*-0.023655}" rpy="0 0 0"/>
   <parent link="${prefix}_calf-motor-driver-ext_1"/>
   <child link="${prefix}_290mm-tie-rod_v1_1"/>
   <axis xyz="0.004243 -0.173596 -0.984808"/>
-  <limit upper="${PI}" lower="${-PI}" velocity="10.0" effort="100.0"/>
 </joint>
 <!-- <joint name="${prefix}_Revolute113" type="revolute">
@@ -2837,6 +2821,6 @@
         <child>${prefix}_thigh-bracket_1</child>
     </joint>
-  <joint name="${prefix}_Revolute71gz" type="revolute">
-          <pose relative_to="${prefix}_double-bracket-10deg_MIR_MIR_MIR_1">-0.06009 -0.001384 ${sign*0.0} 0 0 0</pose>
+    <joint name="${prefix}_Revolute71gz" type="revolute">
+          <pose relative_to="${prefix}_double-bracket-10deg_MIR_MIR_MIR_1">-0.06009 -0.001384 ${sign*-0.007} 0 0 0</pose>
           <parent>${prefix}_double-bracket-10deg_MIR_MIR_MIR_1</parent>
           <child>${prefix}_skateboard-bearing__17__1</child>
@@ -2844,14 +2828,4 @@
               <xyz> 0 0 1</xyz>
           </axis>
-          <limit>
-              <lower>${-PI}</lower>
-              <upper>${PI}</upper>
-              <effort>10.0</effort>
-              <velocity>10.0</velocity>
-          </limit>
-          <!-- <dynamics>
-              <damping>10.0</damping>
-              <friction>0.1</friction>
-          </dynamics> -->
       </joint>
     <joint name="${prefix}_Revolute72gz" type="revolute">
@@ -2862,14 +2836,4 @@
             <xyz> 0 0 1</xyz>
         </axis>
-        <limit>
-            <lower>${-PI}</lower>
-            <upper>${PI}</upper>
-            <effort>10.0</effort>
-            <velocity>10.0</velocity>
-        </limit>
-        <!-- <dynamics>
-            <damping>10.0</damping>
-            <friction>0.1</friction>
-        </dynamics> -->
     </joint>
     <joint name="${prefix}_Revolute73gz" type="revolute">
@@ -2880,14 +2844,4 @@
             <xyz> 0 0 1</xyz>
         </axis>
-        <limit>
-            <lower>${-PI}</lower>
-            <upper>${PI}</upper>
-            <effort>10.0</effort>
-            <velocity>10.0</velocity>
-        </limit>
-        <!-- <dynamics>
-            <damping>10.0</damping>
-            <friction>0.1</friction>
-        </dynamics> -->
     </joint>
     <joint name="${prefix}_Revolute113gz" type="revolute">
@@ -2898,14 +2852,4 @@
             <xyz> 0 0 1</xyz>
         </axis>
-        <limit>
-            <lower>${-PI}</lower>
-            <upper>${PI}</upper>
-            <effort>10.0</effort>
-            <velocity>10.0</velocity>
-        </limit>
-        <!-- <dynamics>
-            <damping>10.0</damping>
-            <friction>0.10</friction>
-        </dynamics> -->
     </joint>
     <joint name="${prefix}_Revolute114gz" type="revolute">
@@ -2916,14 +2860,4 @@
             <xyz> 0 0 1</xyz>
         </axis>
-        <limit>
-            <lower>${-PI}</lower>
-            <upper>${PI}</upper>
-            <effort>10.0</effort>
-            <velocity>10.0</velocity>
-        </limit>
-        <!-- <dynamics>
-            <damping>0.0</damping>
-            <friction>0.0</friction>
-        </dynamics> -->
     </joint>
 </gazebo>

Commit message: Refactor leg.xacro: comment out base link and revolute joint for clarity, adjust joint poses for improved functionality

File: hyperspawn_dropbear_description/urdf/leg.xacro (robot description, xacro)
@@ -2,5 +2,5 @@
 <robot name="humanoidrightleg" xmlns:xacro="http://www.ros.org/wiki/xacro">
   <xacro:macro name="leg_macro" params="prefix folder parent sign *origin">
-<link name="${prefix}_base_link">
+<!-- <link name="${prefix}_base_link">
   <inertial>
     <origin xyz="-2.137404171899072e-14 0 ${sign*0.005}" rpy="0 0 0"/>
@@ -21,5 +21,5 @@
     </geometry>
   </collision>
-</link>
+</link> -->
 <link name="${prefix}_RMD-X10-S2_MIR4__3_Stator_1">
   <inertial>
@@ -2807,10 +2807,10 @@
 <gazebo>
     <joint name="${prefix}_Rigid46gz" type="fixed">
-        <pose relative_to="${prefix}_skateboard-bearing__14__1">-0.01038 0.04119 ${sign*0.0} 0 0 0</pose>
+        <pose relative_to="${prefix}_conjstraint-knee-test-oute_MIR_1">0.0 0 0 0 0 0</pose>
         <parent>${prefix}_conjstraint-knee-test-oute_MIR_1</parent>
         <child>${prefix}_skateboard-bearing__11__1</child>
     </joint>
     <joint name="${prefix}_Rigid47gz" type="fixed">
-        <pose relative_to="${prefix}_skateboard-bearing__13__1">0.1 0.04774 ${sign*0.0} 0 0 0 0 0 0</pose>
+        <pose relative_to="${prefix}_conjstraint-knee-test-oute_1">0 0 0 0 0 0</pose>
         <parent>${prefix}_conjstraint-knee-test-oute_1</parent>
         <child>${prefix}_skateboard-bearing__10__1</child>
@@ -2821,5 +2821,5 @@
         <child>${prefix}_thigh-bracket_1</child>
     </joint>
-    <joint name="${prefix}_Revolute71gz" type="revolute">
+    <!-- <joint name="${prefix}_Revolute71gz" type="revolute">
           <pose relative_to="${prefix}_double-bracket-10deg_MIR_MIR_MIR_1">-0.06009 -0.001384 ${sign*-0.007} 0 0 0</pose>
           <parent>${prefix}_double-bracket-10deg_MIR_MIR_MIR_1</parent>
@@ -2828,5 +2828,5 @@
               <xyz> 0 0 1</xyz>
           </axis>
-      </joint>
+      </joint> -->
     <joint name="${prefix}_Revolute72gz" type="revolute">
         <pose relative_to="${prefix}_double-bracket-10deg_MIR_MIR_MIR_1">0.00 0.00 ${sign*-0.02} 0 0 0</pose>
@@ -2838,7 +2838,16 @@
     </joint>
     <joint name="${prefix}_Revolute73gz" type="revolute">
-        <pose relative_to="${prefix}_double-bracket-10deg_MIR_MIR_MIR_1">-0.06009 -0.001384 ${sign*-0.02} 0 0 0</pose>
-        <parent>${prefix}_double-bracket-10deg_MIR_MIR_MIR_1</parent>
-        <child>${prefix}_skateboard-bearing__12__1</child>
+        <pose relative_to="${prefix}_skateboard-bearing__12__1">-0.06009 -0.001384 ${sign*0.02} 0 0 0</pose>
+        <parent>${prefix}_skateboard-bearing__12__1</parent>
+        <child>${prefix}_double-bracket-10deg_MIR_MIR_MIR_1</child>
+        <axis>
+            <xyz> 0 0 1</xyz>
+        </axis>
+    </joint>
+    <joint name="${prefix}_Bearing17_12_Revolutegz" type="revolute">
+        <!-- <pose relative_to="${prefix}_skateboard-bearing__12__1">-0.012 0.02561 ${sign*0.01} 0 0 0</pose> -->
+        <pose relative_to="${prefix}_skateboard-bearing__12__1">0.025 -0.05433 ${sign*-0.01} 0 0 0</pose>
+        <parent>${prefix}_skateboard-bearing__12__1</parent>
+        <child>${prefix}_skateboard-bearing__17__1</child>
         <axis>
             <xyz> 0 0 1</xyz>

Commit message: Uncomment joint definitions in leg.xacro for improved robot joint configuration

File: hyperspawn_dropbear_description/urdf/leg.xacro (robot description, xacro)
@@ -2821,5 +2821,5 @@
         <child>${prefix}_thigh-bracket_1</child>
     </joint>
-    <!-- <joint name="${prefix}_Revolute71gz" type="revolute">
+    <joint name="${prefix}_Revolute71gz" type="revolute">
           <pose relative_to="${prefix}_double-bracket-10deg_MIR_MIR_MIR_1">-0.06009 -0.001384 ${sign*-0.007} 0 0 0</pose>
           <parent>${prefix}_double-bracket-10deg_MIR_MIR_MIR_1</parent>
@@ -2828,5 +2828,5 @@
               <xyz> 0 0 1</xyz>
           </axis>
-      </joint> -->
+      </joint>
     <joint name="${prefix}_Revolute72gz" type="revolute">
         <pose relative_to="${prefix}_double-bracket-10deg_MIR_MIR_MIR_1">0.00 0.00 ${sign*-0.02} 0 0 0</pose>
@@ -2841,13 +2841,4 @@
         <parent>${prefix}_skateboard-bearing__12__1</parent>
         <child>${prefix}_double-bracket-10deg_MIR_MIR_MIR_1</child>
-        <axis>
-            <xyz> 0 0 1</xyz>
-        </axis>
-    </joint>
-    <joint name="${prefix}_Bearing17_12_Revolutegz" type="revolute">
-        <!-- <pose relative_to="${prefix}_skateboard-bearing__12__1">-0.012 0.02561 ${sign*0.01} 0 0 0</pose> -->
-        <pose relative_to="${prefix}_skateboard-bearing__12__1">0.025 -0.05433 ${sign*-0.01} 0 0 0</pose>
-        <parent>${prefix}_skateboard-bearing__12__1</parent>
-        <child>${prefix}_skateboard-bearing__17__1</child>
         <axis>
             <xyz> 0 0 1</xyz>
