Commit message: Replace material "opaque2550255" with "steel_satin" in materials.xacro for improved visual representation.

File: humanoidrightarm_description/urdf/humanoidrightarm.xacro (robot description, xacro)
@@ -5,7 +5,7 @@
 <link name="base_link">
   <inertial>
-    <origin xyz="-4.564684959507811e-14 -1.297744842251468e-14 -0.00040000000000051" rpy="0 0 0"/>
-    <mass value="0.0710251267123582"/>
-    <inertia ixx="1.03755872605632e-05" iyy="1.03755872605639e-05" izz="2.04552364931589e-05" ixy="2.231104194494098e-20" iyz="-3.993969333038147e-17" ixz="8.809863505376990e-17"/>
+    <origin xyz="-6.496817022290221e-15 0 0.005" rpy="0 0 0"/>
+    <mass value="0.49623462441733"/>
+    <inertia ixx="0.000272043421613551" iyy="0.000272043421603598" izz="0.000535816266143527" ixy="-8.924416761146857e-20" iyz="0" ixz="3.081487911019577e-33"/>
   </inertial>
   <visual>
@@ -14,5 +14,5 @@
       <mesh filename="package://humanoidrightarm_description/meshes/base_link.stl" scale="0.001 0.001 0.001"/>
     </geometry>
-    <material name="opaque2550255"/>
+    <material name="steel_satin"/>
   </visual>
   <collision>
@@ -23,12 +23,1332 @@
   </collision>
 </link>
+<link name="shoulder-roll-al-mot_MIR1__1__1">
+  <inertial>
+    <origin xyz="-0.01659232442569455 1.1139623568467982e-07 0.013349013943229465" rpy="0 0 0"/>
+    <mass value="0.0163592682580457"/>
+    <inertia ixx="2.94469554646068e-06" iyy="1.41414366306325e-06" izz="2.28526048528149e-06" ixy="-1.959109032158722e-11" iyz="3.686440548058393e-11" ixz="1.74158424577829e-08"/>
+  </inertial>
+  <visual>
+    <origin xyz="-0.0 -0.0 -0.01" rpy="0 0 0"/>
+    <geometry>
+      <mesh filename="package://humanoidrightarm_description/meshes/shoulder-roll-al-mot_MIR1__1__1.stl" scale="0.001 0.001 0.001"/>
+    </geometry>
+    <material name="opaque245245245"/>
+  </visual>
+  <collision>
+    <origin xyz="-0.0 -0.0 -0.01" rpy="0 0 0"/>
+    <geometry>
+      <mesh filename="package://humanoidrightarm_description/meshes/shoulder-roll-al-mot_MIR1__1__1.stl" scale="0.001 0.001 0.001"/>
+    </geometry>
+  </collision>
+</link>
+<link name="shoulder-roll-al-mot_MIR1__2__1">
+  <inertial>
+    <origin xyz="0.016592324425693906 -1.1139623519396125e-07 0.013349013943229461" rpy="0 0 0"/>
+    <mass value="0.0163592682580457"/>
+    <inertia ixx="2.94469554646068e-06" iyy="1.41414366306325e-06" izz="2.2852604852815e-06" ixy="-1.959109029246965e-11" iyz="-3.686440548014597e-11" ixz="-1.74158424577846e-08"/>
+  </inertial>
+  <visual>
+    <origin xyz="-0.0 -0.0 -0.01" rpy="0 0 0"/>
+    <geometry>
+      <mesh filename="package://humanoidrightarm_description/meshes/shoulder-roll-al-mot_MIR1__2__1.stl" scale="0.001 0.001 0.001"/>
+    </geometry>
+    <material name="opaque245245245"/>
+  </visual>
+  <collision>
+    <origin xyz="-0.0 -0.0 -0.01" rpy="0 0 0"/>
+    <geometry>
+      <mesh filename="package://humanoidrightarm_description/meshes/shoulder-roll-al-mot_MIR1__2__1.stl" scale="0.001 0.001 0.001"/>
+    </geometry>
+  </collision>
+</link>
+<link name="yaw-cap_1">
+  <inertial>
+    <origin xyz="2.2162578884901502e-14 2.2140731002778117e-16 -0.006586829858195156" rpy="0 0 0"/>
+    <mass value="0.017312584943862"/>
+    <inertia ixx="5.04854323001019e-06" iyy="2.6638750836575e-06" izz="3.35018570940257e-06" ixy="1.908869042176979e-20" iyz="1.100622863726450e-19" ixz="3.662235970160196e-18"/>
+  </inertial>
+  <visual>
+    <origin xyz="-0.0 -0.0 -0.11" rpy="0 0 0"/>
+    <geometry>
+      <mesh filename="package://humanoidrightarm_description/meshes/yaw-cap_1.stl" scale="0.001 0.001 0.001"/>
+    </geometry>
+    <material name="opaque245245245"/>
+  </visual>
+  <collision>
+    <origin xyz="-0.0 -0.0 -0.11" rpy="0 0 0"/>
+    <geometry>
+      <mesh filename="package://humanoidrightarm_description/meshes/yaw-cap_1.stl" scale="0.001 0.001 0.001"/>
+    </geometry>
+  </collision>
+</link>
+<link name="yaw-waist-adapter-motor-exal_MIR1_1">
+  <inertial>
+    <origin xyz="0.00723403458529202 -3.5971225997855074e-16 0.0499999999999884" rpy="0 0 0"/>
+    <mass value="0.0437734881347393"/>
+    <inertia ixx="1.66949657418105e-05" iyy="8.2583522562858e-06" izz="1.50911001770001e-05" ixy="-2.786381389588518e-20" iyz="-1.216427996016598e-20" ixz="-2.236166980751353e-19"/>
+  </inertial>
+  <visual>
+    <origin xyz="-0.0 -0.0 -0.01" rpy="0 0 0"/>
+    <geometry>
+      <mesh filename="package://humanoidrightarm_description/meshes/yaw-waist-adapter-motor-exal_MIR1_1.stl" scale="0.001 0.001 0.001"/>
+    </geometry>
+    <material name="opaque245245245"/>
+  </visual>
+  <collision>
+    <origin xyz="-0.0 -0.0 -0.01" rpy="0 0 0"/>
+    <geometry>
+      <mesh filename="package://humanoidrightarm_description/meshes/yaw-waist-adapter-motor-exal_MIR1_1.stl" scale="0.001 0.001 0.001"/>
+    </geometry>
+  </collision>
+</link>
+<link name="front-bearing-adapter-shoulder_1">
+  <inertial>
+    <origin xyz="0.007601634210069975 -0.015587999999998516 -0.00900000000001975" rpy="0 0 0"/>
+    <mass value="0.0277092360547985"/>
+    <inertia ixx="8.78070443423959e-06" iyy="3.7939788402805e-06" izz="6.10989221729227e-06" ixy="3.877429965353465e-20" iyz="-1.823094394463676e-20" ixz="1.219727444046192e-18"/>
+  </inertial>
+  <visual>
+    <origin xyz="-0.02 -0.015588 -0.069" rpy="0 0 0"/>
+    <geometry>
+      <mesh filename="package://humanoidrightarm_description/meshes/front-bearing-adapter-shoulder_1.stl" scale="0.001 0.001 0.001"/>
+    </geometry>
+    <material name="opaque191191191"/>
+  </visual>
+  <collision>
+    <origin xyz="-0.02 -0.015588 -0.069" rpy="0 0 0"/>
+    <geometry>
+      <mesh filename="package://humanoidrightarm_description/meshes/front-bearing-adapter-shoulder_1.stl" scale="0.001 0.001 0.001"/>
+    </geometry>
+  </collision>
+</link>
+<link name="shoulder-ex-al-interface__2__1">
+  <inertial>
+    <origin xyz="-0.008272088271638172 -0.015588000000004406 -0.008999999999990647" rpy="0 0 0"/>
+    <mass value="0.03263560284613"/>
+    <inertia ixx="1.03830779561817e-05" iyy="4.49807884871569e-06" izz="7.37834772831807e-06" ixy="2.358671083983723e-19" iyz="-9.132545078240102e-17" ixz="6.844026213814747e-19"/>
+  </inertial>
+  <visual>
+    <origin xyz="0.01 -0.015588 -0.069" rpy="0 0 0"/>
+    <geometry>
+      <mesh filename="package://humanoidrightarm_description/meshes/shoulder-ex-al-interface__2__1.stl" scale="0.001 0.001 0.001"/>
+    </geometry>
+    <material name="opaque22122113"/>
+  </visual>
+  <collision>
+    <origin xyz="0.01 -0.015588 -0.069" rpy="0 0 0"/>
+    <geometry>
+      <mesh filename="package://humanoidrightarm_description/meshes/shoulder-ex-al-interface__2__1.stl" scale="0.001 0.001 0.001"/>
+    </geometry>
+  </collision>
+</link>
+<link name="RMD-X8-Pro_MIR8_MIR1__1__1">
+  <inertial>
+    <origin xyz="-0.02188091903208703 -3.219454781594442e-06 0.0004617607023024439" rpy="0 0 0"/>
+    <mass value="0.780215846180861"/>
+    <inertia ixx="0.00111113799843006" iyy="0.000764684770745232" izz="0.000752808817666897" ixy="4.74278772872876e-08" iyz="-2.07243316667861e-08" ixz="8.89585651039351e-06"/>
+  </inertial>
+  <visual>
+    <origin xyz="0.027 0.0 -0.06" rpy="0 0 0"/>
+    <geometry>
+      <mesh filename="package://humanoidrightarm_description/meshes/RMD-X8-Pro_MIR8_MIR1__1__1.stl" scale="0.001 0.001 0.001"/>
+    </geometry>
+    <material name="opaque13110895"/>
+  </visual>
+  <collision>
+    <origin xyz="0.027 0.0 -0.06" rpy="0 0 0"/>
+    <geometry>
+      <mesh filename="package://humanoidrightarm_description/meshes/RMD-X8-Pro_MIR8_MIR1__1__1.stl" scale="0.001 0.001 0.001"/>
+    </geometry>
+  </collision>
+</link>
+<link name="shoulder-motor-bicep-rotor-bracket_1">
+  <inertial>
+    <origin xyz="-0.005500000000001365 -0.010394566089843876 0.006894585665480776" rpy="0 0 0"/>
+    <mass value="0.0283879289585321"/>
+    <inertia ixx="1.23170131575466e-05" iyy="8.18018047261162e-06" izz="4.70932258559873e-06" ixy="-1.355252715606881e-19" iyz="1.60448646361674e-06" ixz="5.421010862427522e-20"/>
+  </inertial>
+  <visual>
+    <origin xyz="0.0645 0.042 -0.06" rpy="0 0 0"/>
+    <geometry>
+      <mesh filename="package://humanoidrightarm_description/meshes/shoulder-motor-bicep-rotor-bracket_1.stl" scale="0.001 0.001 0.001"/>
+    </geometry>
+    <material name="opaque245245245"/>
+  </visual>
+  <collision>
+    <origin xyz="0.0645 0.042 -0.06" rpy="0 0 0"/>
+    <geometry>
+      <mesh filename="package://humanoidrightarm_description/meshes/shoulder-motor-bicep-rotor-bracket_1.stl" scale="0.001 0.001 0.001"/>
+    </geometry>
+  </collision>
+</link>
+<link name="bicep-rear-motor-adapter_1">
+  <inertial>
+    <origin xyz="0.015923392949308564 -0.003183487341080926 0.0155000000000022" rpy="0 0 0"/>
+    <mass value="0.0329567035250635"/>
+    <inertia ixx="5.38963285566697e-06" iyy="8.54909107225949e-06" izz="7.46209316246797e-06" ixy="-7.58704318227122e-07" iyz="2.710505431213761e-20" ixz="1.626303258728257e-19"/>
+  </inertial>
+  <visual>
+    <origin xyz="0.0645 0.06 -0.0585" rpy="0 0 0"/>
+    <geometry>
+      <mesh filename="package://humanoidrightarm_description/meshes/bicep-rear-motor-adapter_1.stl" scale="0.001 0.001 0.001"/>
+    </geometry>
+    <material name="opaque191191191"/>
+  </visual>
+  <collision>
+    <origin xyz="0.0645 0.06 -0.0585" rpy="0 0 0"/>
+    <geometry>
+      <mesh filename="package://humanoidrightarm_description/meshes/bicep-rear-motor-adapter_1.stl" scale="0.001 0.001 0.001"/>
+    </geometry>
+  </collision>
+</link>
+<link name="bicep-shoulder-bracket-exal__1__1">
+  <inertial>
+    <origin xyz="-0.00799999999999938 -0.009999999999990211 0.005535150009386841" rpy="0 0 0"/>
+    <mass value="0.0139230350925919"/>
+    <inertia ixx="1.84871225007599e-06" iyy="1.17647287887655e-06" izz="2.74606964176384e-06" ixy="-4.065758146820642e-20" iyz="-2.710505431213761e-20" ixz="-6.776263578034403e-21"/>
+  </inertial>
+  <visual>
+    <origin xyz="0.0265 0.06 -0.084" rpy="0 0 0"/>
+    <geometry>
+      <mesh filename="package://humanoidrightarm_description/meshes/bicep-shoulder-bracket-exal__1__1.stl" scale="0.001 0.001 0.001"/>
+    </geometry>
+    <material name="opaque245245245"/>
+  </visual>
+  <collision>
+    <origin xyz="0.0265 0.06 -0.084" rpy="0 0 0"/>
+    <geometry>
+      <mesh filename="package://humanoidrightarm_description/meshes/bicep-shoulder-bracket-exal__1__1.stl" scale="0.001 0.001 0.001"/>
+    </geometry>
+  </collision>
+</link>
+<link name="bicep-shoulder-bracket-exal__2__1">
+  <inertial>
+    <origin xyz="-0.00799999999999845 -0.009999999999987075 -0.005464849990612884" rpy="0 0 0"/>
+    <mass value="0.0139230350925919"/>
+    <inertia ixx="1.84871225007599e-06" iyy="1.17647287887658e-06" izz="2.74606964176389e-06" ixy="-4.065758146820642e-20" iyz="-2.032879073410321e-20" ixz="-6.776263578034403e-21"/>
+  </inertial>
+  <visual>
+    <origin xyz="0.0265 0.06 -0.064" rpy="0 0 0"/>
+    <geometry>
+      <mesh filename="package://humanoidrightarm_description/meshes/bicep-shoulder-bracket-exal__2__1.stl" scale="0.001 0.001 0.001"/>
+    </geometry>
+    <material name="opaque245245245"/>
+  </visual>
+  <collision>
+    <origin xyz="0.0265 0.06 -0.064" rpy="0 0 0"/>
+    <geometry>
+      <mesh filename="package://humanoidrightarm_description/meshes/bicep-shoulder-bracket-exal__2__1.stl" scale="0.001 0.001 0.001"/>
+    </geometry>
+  </collision>
+</link>
+<link name="2020_100mm__8___1__1">
+  <inertial>
+    <origin xyz="0.03999999999997527 0.009999999999997691 -0.009999999999981204" rpy="0 0 0"/>
+    <mass value="0.0528977181003175"/>
+    <inertia ixx="4.31100866363557e-06" iyy="4.62369360821583e-05" izz="4.62369360817191e-05" ixy="-4.940218111474687e-17" iyz="1.084202172485504e-19" ixz="-2.516514389746603e-17"/>
+  </inertial>
+  <visual>
+    <origin xyz="0.04 0.09 -0.084" rpy="0 0 0"/>
+    <geometry>
+      <mesh filename="package://humanoidrightarm_description/meshes/2020_100mm__8___1__1.stl" scale="0.001 0.001 0.001"/>
+    </geometry>
+    <material name="opaque727161"/>
+  </visual>
+  <collision>
+    <origin xyz="0.04 0.09 -0.084" rpy="0 0 0"/>
+    <geometry>
+      <mesh filename="package://humanoidrightarm_description/meshes/2020_100mm__8___1__1.stl" scale="0.001 0.001 0.001"/>
+    </geometry>
+  </collision>
+</link>
+<link name="yaw-waist-adapter-motor-exal_MIR1__5__1">
+  <inertial>
+    <origin xyz="-0.04999999999998893 0.007234034585292329 2.0539125955565396e-15" rpy="0 0 0"/>
+    <mass value="0.0437734881347393"/>
+    <inertia ixx="1.50911001770002e-05" iyy="1.66949657418102e-05" izz="8.25835225628604e-06" ixy="1.712452913172996e-19" iyz="2.710505431213761e-20" ixz="-1.982913302373183e-20"/>
+  </inertial>
+  <visual>
+    <origin xyz="-0.05 0.08 -0.074" rpy="0 0 0"/>
+    <geometry>
+      <mesh filename="package://humanoidrightarm_description/meshes/yaw-waist-adapter-motor-exal_MIR1__5__1.stl" scale="0.001 0.001 0.001"/>
+    </geometry>
+    <material name="opaque245245245"/>
+  </visual>
+  <collision>
+    <origin xyz="-0.05 0.08 -0.074" rpy="0 0 0"/>
+    <geometry>
+      <mesh filename="package://humanoidrightarm_description/meshes/yaw-waist-adapter-motor-exal_MIR1__5__1.stl" scale="0.001 0.001 0.001"/>
+    </geometry>
+  </collision>
+</link>
+<link name="bicep-shoulder-bracket-exal_1">
+  <inertial>
+    <origin xyz="-0.01550000000000154 0.020000000000012313 -0.007214849990613059" rpy="0 0 0"/>
+    <mass value="0.0139230350925919"/>
+    <inertia ixx="1.84871225007598e-06" iyy="1.17647287887656e-06" izz="2.74606964176393e-06" ixy="-3.388131789017201e-20" iyz="-1.355252715606881e-20" ixz="0"/>
+  </inertial>
+  <visual>
+    <origin xyz="-0.05 0.09 -0.06575" rpy="0 0 0"/>
+    <geometry>
+      <mesh filename="package://humanoidrightarm_description/meshes/bicep-shoulder-bracket-exal_1.stl" scale="0.001 0.001 0.001"/>
+    </geometry>
+    <material name="opaque245245245"/>
+  </visual>
+  <collision>
+    <origin xyz="-0.05 0.09 -0.06575" rpy="0 0 0"/>
+    <geometry>
+      <mesh filename="package://humanoidrightarm_description/meshes/bicep-shoulder-bracket-exal_1.stl" scale="0.001 0.001 0.001"/>
+    </geometry>
+  </collision>
+</link>
+<link name="shoulder-front_1">
+  <inertial>
+    <origin xyz="-0.007736652232246094 0.010361414448293069 0.010000000000001535" rpy="0 0 0"/>
+    <mass value="0.0334504701906665"/>
+    <inertia ixx="6.75301171017896e-06" iyy="6.11839158981428e-06" izz="5.9732489883625e-06" ixy="-6.72891148221279e-08" iyz="1.539024983843174e-16" ixz="-6.640738306473715e-19"/>
+  </inertial>
+  <visual>
+    <origin xyz="-0.0425 0.06 -0.064" rpy="0 0 0"/>
+    <geometry>
+      <mesh filename="package://humanoidrightarm_description/meshes/shoulder-front_1.stl" scale="0.001 0.001 0.001"/>
+    </geometry>
+    <material name="opaque191191191"/>
+  </visual>
+  <collision>
+    <origin xyz="-0.0425 0.06 -0.064" rpy="0 0 0"/>
+    <geometry>
+      <mesh filename="package://humanoidrightarm_description/meshes/shoulder-front_1.stl" scale="0.001 0.001 0.001"/>
+    </geometry>
+  </collision>
+</link>
+<link name="bicep-shoulder-bracket-exal__3__1">
+  <inertial>
+    <origin xyz="-0.008000000000001208 -0.00999999999998867 0.005535150009387327" rpy="0 0 0"/>
+    <mass value="0.0139230350925919"/>
+    <inertia ixx="1.84871225007602e-06" iyy="1.1764728788765e-06" izz="2.74606964176393e-06" ixy="-4.065758146820642e-20" iyz="-4.065758146820642e-20" ixz="-6.776263578034403e-21"/>
+  </inertial>
+  <visual>
+    <origin xyz="-0.0425 0.06 -0.084" rpy="0 0 0"/>
+    <geometry>
+      <mesh filename="package://humanoidrightarm_description/meshes/bicep-shoulder-bracket-exal__3__1.stl" scale="0.001 0.001 0.001"/>
+    </geometry>
+    <material name="opaque245245245"/>
+  </visual>
+  <collision>
+    <origin xyz="-0.0425 0.06 -0.084" rpy="0 0 0"/>
+    <geometry>
+      <mesh filename="package://humanoidrightarm_description/meshes/bicep-shoulder-bracket-exal__3__1.stl" scale="0.001 0.001 0.001"/>
+    </geometry>
+  </collision>
+</link>
+<link name="shoulder-cap_1">
+  <inertial>
+    <origin xyz="0.004917614424534554 0.03505255276075949 -0.025722563916740007" rpy="0 0 0"/>
+    <mass value="0.0540863834696359"/>
+    <inertia ixx="4.35959437594329e-05" iyy="1.82034440516574e-05" izz="2.63665724286844e-05" ixy="3.09573929524443e-08" iyz="4.95302874574802e-06" ixz="-1.46040514440132e-08"/>
+  </inertial>
+  <visual>
+    <origin xyz="-0.05 0.042 -0.089" rpy="0 0 0"/>
+    <geometry>
+      <mesh filename="package://humanoidrightarm_description/meshes/shoulder-cap_1.stl" scale="0.001 0.001 0.001"/>
+    </geometry>
+    <material name="opaque245245245"/>
+  </visual>
+  <collision>
+    <origin xyz="-0.05 0.042 -0.089" rpy="0 0 0"/>
+    <geometry>
+      <mesh filename="package://humanoidrightarm_description/meshes/shoulder-cap_1.stl" scale="0.001 0.001 0.001"/>
+    </geometry>
+  </collision>
+</link>
+<link name="shoulder-front-bearing-adapter_1">
+  <inertial>
+    <origin xyz="-0.007720854302206356 1.4675767796906362e-15 -2.1421753260142395e-13" rpy="0 0 0"/>
+    <mass value="0.060585838929716"/>
+    <inertia ixx="4.09629608015188e-05" iyy="2.1661885549037e-05" izz="2.16618856541457e-05" ixy="2.751034531088321e-19" iyz="7.982245490983458e-20" ixz="-2.710505431213761e-19"/>
+  </inertial>
+  <visual>
+    <origin xyz="-0.05 -0.0 -0.06" rpy="0 0 0"/>
+    <geometry>
+      <mesh filename="package://humanoidrightarm_description/meshes/shoulder-front-bearing-adapter_1.stl" scale="0.001 0.001 0.001"/>
+    </geometry>
+    <material name="opaque22122113"/>
+  </visual>
+  <collision>
+    <origin xyz="-0.05 -0.0 -0.06" rpy="0 0 0"/>
+    <geometry>
+      <mesh filename="package://humanoidrightarm_description/meshes/shoulder-front-bearing-adapter_1.stl" scale="0.001 0.001 0.001"/>
+    </geometry>
+  </collision>
+</link>
+<link name="skateboard-bearing__7__1">
+  <inertial>
+    <origin xyz="-0.003500427124746859 9.925393840148899e-16 6.552397513459596e-14" rpy="0 0 0"/>
+    <mass value="0.00270161260245453"/>
+    <inertia ixx="1.85060463480797e-07" iyy="1.03561816321086e-07" izz="1.0356181674642e-07" ixy="7.325440669930568e-22" iyz="-9.492407324726906e-23" ixz="8.470329472543003e-22"/>
+  </inertial>
+  <visual>
+    <origin xyz="-0.046172 -0.0 -0.06" rpy="0 0 0"/>
+    <geometry>
+      <mesh filename="package://humanoidrightarm_description/meshes/skateboard-bearing__7__1.stl" scale="0.001 0.001 0.001"/>
+    </geometry>
+    <material name="opaque191191191"/>
+  </visual>
+  <collision>
+    <origin xyz="-0.046172 -0.0 -0.06" rpy="0 0 0"/>
+    <geometry>
+      <mesh filename="package://humanoidrightarm_description/meshes/skateboard-bearing__7__1.stl" scale="0.001 0.001 0.001"/>
+    </geometry>
+  </collision>
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
File: humanoidrightarm_description/urdf/materials.xacro (robot description, xacro)
@@ -28,6 +28,6 @@
   <color rgba="0.5137254901960784 0.4235294117647059 0.37254901960784315 1.0"/>
 </material>
-<material name="opaque2550255">
-  <color rgba="1.0 0.0 1.0 1.0"/>
+<material name="steel_satin">
+  <color rgba="0.6274509803921569 0.6274509803921569 0.6274509803921569 1.0"/>
 </material>
 </robot>
